File: wa_psu.sch (EAGLE design)
At the start: 38 parts, among them Q1 SI7489DP, Q2 CPH3459, U1 LMV7219, U2 LM2936

Commit message: Work on the PSU
Parts:
- added U$10, U$9: DCDC 15V, ICs:PDQE10-Q48-S15
- added U$8: DCDC +/-15V, ICs:PDQE10-Q48-D15-D
Changed lines of the file:
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@@
 <part name="GND18" library="NETS" deviceset="GND" device=""/>
 <part name="U$7" library="NETS" deviceset="VOUT" device=""/>
+<part name="U$8" library="ICs" deviceset="PDQE10-Q48-D15-D" device="" value="DCDC +/-15V"/>
+<part name="U$9" library="ICs" deviceset="PDQE10-Q48-S15" device="" value="DCDC 15V"/>
+<part name="U$10" library="ICs" deviceset="PDQE10-Q48-S15" device="" value="DCDC 15V"/>
 </parts>
 <sheets>
@@
 <attribute name="VALUE" x="406.4" y="116.84" size="1.778" layer="96" rot="R180" align="center"/>
 </instance>
+<instance part="U$8" gate="G$1" x="375.92" y="17.78" smashed="yes">
+<attribute name="NAME" x="368.3" y="40.64" size="1.778" layer="95"/>
+<attribute name="VALUE" x="368.3" y="38.1" size="1.778" layer="95"/>
+</instance>
+<instance part="U$9" gate="G$1" x="378.46" y="-63.5" smashed="yes">
+<attribute name="NAME" x="370.84" y="-40.64" size="1.778" layer="95"/>
+<attribute name="VALUE" x="370.84" y="-43.18" size="1.778" layer="95"/>
+</instance>
+<instance part="U$10" gate="G$1" x="373.38" y="-149.86" smashed="yes">
+<attribute name="NAME" x="365.76" y="-127" size="1.778" layer="95"/>
+<attribute name="VALUE" x="365.76" y="-129.54" size="1.778" layer="95"/>
+</instance>
 </instances>

Commit message: Ready for layout
Parts:
- removed U$10, U$9: DCDC 15V, ICs:PDQE10-Q48-S15
- removed U$8: DCDC +/-15V, ICs:PDQE10-Q48-D15-D
- added C11, C12, C13, C14, C17: 25V 1000uF, CAPACITORS:25ZLJ1000M10X20
- added C15, C16: 1uF 25V, CAPACITORS:CL10A105KA8NNNC
- added L5, L6, L7, L8: 470uH, INDUCTORS:SRN1060-471M
- added Q3: SI4848ADY, TRANSISTORs:SI4848ADY-T1-GE3
- added R13: 10k, r_0603:ERJ3EKF1002V
- added R14: 100R, RESISTORS:ERG-3SJ101V
- added R15: 240R, r_0603:ERJ3EKF2400V
- added R16: 2.0k, r_0603:ERJ3EKF2001V
- added U3: DCDC +/-15V, ICs:PDQE10-Q48-D15-D
- added U4, U5: DCDC 15V, ICs:PDQE10-Q48-S15
- added U6: LM317, ICs:LM317T
Connections:
- removed net N$10: L3.2, L4.1
- new net AMP_12V: C16.2, C17.A, R15.2, U6.VOUT
- new net DSP_AGND: C11.K, C12.A, U3.COM
- new net DSP_DGND: C13.K, U4.COM
- new net DSP_VA+: C11.A, L5.2
- new net DSP_VA-: C12.K, L6.2
- new net DSP_VD+: C13.A, L7.2
- new net N$12: L5.1, U3.VO+
- new net N$13: L6.1, U3.VO-
- new net N$14: R15.1, R16.2, U6.ADJ
- new net N$18: C14.A, C15.2, L8.2, U6.VIN
- new net N$20: L8.1, U5.VO+
- new net N$22: L7.1, U4.VO+
- new net N$23: Q3.D, R14.1
- new net PGND: C14.K, C15.1, C16.1, C17.K, R16.1, U5.COM
- net GND: now also Q3.S, R13.1, U3.VIN-, U4.VIN-, U5.VIN-
- net N$4: now also L3.2, L4.1
- net PSU_VIN_OVERVOLT: now also Q3.G, R13.2
- net VIN: now also R14.2, U3.VIN+, U4.VIN+, U5.VIN+
Other:
- moved on the sheet: C1, C10, C2, C3, C4, C5, C6, C7, C8, C9, D1, D2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

Commit message: Layout nearly complete
Parts:
- added C18: 100nF 16V, CAPACITORS:CL10B104KO8WPNC
- added HOLE1, HOLE2, HOLE3, HOLE4, HOLE5, HOLE6, HOLE7, HOLE8: 4mm ID, MISC:MOUNTHOLE_METAL
- added HOLE10, HOLE11, HOLE12, HOLE13, HOLE14, HOLE9: MOUNTHOLE_METAL4X2, MISC:MOUNTHOLE_METAL4X2
- added MECH1, MECH2, MECH3, MECH4: 6mm x 3mm, MISC:MOUNTHOLE
- added R17: 100k, r_0603:ERJ3EKF1003V
- R20: device r_0402:ERJ-2RKF1001X -> r_0603:ERJ3EKF1001V
Connections:
- net 5V: now also C18.2
- net AMP_12V: now also HOLE10.1, HOLE12.1, HOLE14.1
- net GND: now also C18.1, HOLE2.1, HOLE3.1, HOLE5.1, HOLE7.1
- net N$1: now also C1.2, HOLE1.1
- net N$3: now also R17.2
- net N$8: now also R17.1; no longer C1.2
- net PGND: now also HOLE11.1, HOLE13.1, HOLE9.1
- net VOUT: now also HOLE4.1, HOLE6.1, HOLE8.1
Other:
- moved on the sheet: C1, Q2, R1, R2
