File: wa_amp.sch (EAGLE design)
At the start: 89 parts, among them U4 TPA3255, U5 LME49720, U6 LME49720

Commit message: Work on the amplifier
Parts:
- removed C68, C69, C72, C73: 100nF 16V, CAPACITORS:CL10B104KO8WPNC
- removed C70, C71, C74, C75: 330pF 50V, CAPACITORS:CC0603JRNPO9BN331
- removed R37, R38, R39, R40, R41, R42, R43, R44: 10k, r_0603:ERJ3EKF1002V
- removed U5, U6: LME49720, ICs:LME49720MA/NOPB
- added HOLE1, HOLE2, HOLE3, HOLE4: MOUNTHOLE_METAL6X3, MISC:MOUNTHOLE_METAL6X3
- added MECH1, MECH2, MECH3, MECH4: 6mm x 3mm, MISC:MOUNTHOLE
- added TP1, TP2, TP3, TP4, TP5, TP6, TP7, TP8: 2MM_TEST_POINT, MISC:2MM_TEST_POINT
Connections:
- removed net 5VA+: C68.2, C72.2, U5A.V+, U6A.V+
- removed net 5VA-: C69.2, C73.2, U5A.V-, U6A.V-
- removed net N$65: C70.2, R34.1, R38.1, R39.2, U5A.OUT
- removed net N$66: C70.1, R37.1, R38.2, U5A.-
- removed net N$67: R37.2
- removed net N$68: C71.2, R40.1, R45.1, U5B.OUT
- removed net N$69: C71.1, R39.1, R40.2, U5B.-
- removed net N$70: C74.2, R42.1, R43.2, R46.1, U6A.OUT
- removed net N$71: C74.1, R41.1, R42.2, U6A.-
- removed net N$72: R41.2
- removed net N$73: C75.2, R44.1, R47.1, U6B.OUT
- removed net N$74: C75.1, R43.1, R44.2, U6B.-
- removed net N$84: C77.1, C83.1, R46.2, R52.1
- new net N$2: C77.1, C81.1, R46.2, R50.1
- new net N$3: R34.1, TP3.P$1
- new net N$4: R45.1, TP5.P$1
- new net N$5: R46.1, TP6.P$1
- new net N$6: R47.1, TP8.P$1
- net 12V: now also TP1.P$1
- net GND: now also TP2.P$1, TP4.P$1, TP7.P$1; no longer C68.1, C69.1, C72.1, C73.1, U5A.+, U5B.+, U6A.+, U6B.+
- net N$63: now also HOLE1.1
- net N$79: now also HOLE2.1
- net N$81: now also C83.1, R52.1; no longer C81.1, R50.1
- net N$82: now also HOLE3.1
- net N$85: now also HOLE4.1
