File: wa_psu.brd (EAGLE design)
At the start: 150 x 150 mm, 38 parts, among them Q1 SI7489DP, Q2 CPH3459, U1 LMV7219, U2 LM2936

Commit message: Work on the PSU
Parts:
- added U$10, U$9: DCDC 15V, ICs:PDQE10
- added U$8: DCDC +/-15V, ICs:PDQE10
Changed lines of the file:
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@@
 <attribute name="NAME" x="-1.175" y="-387.44" size="2" layer="25"/>
+</element>
+<element name="U$8" library="ICs" package="PDQE10" value="DCDC +/-15V" x="-150" y="-300" smashed="yes">
+<attribute name="DIGIKEY" value="102-4868-ND" x="-150" y="-300" size="1.778" layer="27" display="off"/>
+<attribute name="HEIGHT" value="12" x="-150" y="-300" size="1.778" layer="27" display="off"/>
+<attribute name="NAME" x="-162.625" y="-287.125" size="1" layer="21"/>
+<attribute name="PRICE_PER" value="13.64" x="-150" y="-300" size="1.778" layer="27" display="off"/>
+</element>
+<element name="U$9" library="ICs" package="PDQE10" value="DCDC 15V" x="-300" y="-300" smashed="yes">
+<attribute name="DIGIKEY" value="PDQE10-Q48-S15-D" x="-300" y="-300" size="1.778" layer="27" display="off"/>
+<attribute name="HEIGHT" value="12" x="-300" y="-300" size="1.778" layer="27" display="off"/>
+<attribute name="NAME" x="-312.625" y="-287.125" size="1" layer="21"/>
+<attribute name="PRICE_PER" value="12.18" x="-300" y="-300" size="1.778" layer="27" display="off"/>
+</element>
+<element name="U$10" library="ICs" package="PDQE10" value="DCDC 15V" x="-450" y="-300" smashed="yes">
+<attribute name="DIGIKEY" value="PDQE10-Q48-S15-D" x="-450" y="-300" size="1.778" layer="27" display="off"/>
+<attribute name="HEIGHT" value="12" x="-450" y="-300" size="1.778" layer="27" display="off"/>
+<attribute name="NAME" x="-462.625" y="-287.125" size="1" layer="21"/>
+<attribute name="PRICE_PER" value="12.18" x="-450" y="-300" size="1.778" layer="27" display="off"/>
 </element>
 </elements>

Commit message: Ready for layout
Parts:
- removed U$10, U$9: DCDC 15V, ICs:PDQE10
- removed U$8: DCDC +/-15V, ICs:PDQE10
- added C11, C12, C13, C14, C17: 25V 1000uF, CAPACITORS:10MM_RADIAL_5MM_PITCH
- added C15, C16: 1uF 25V, CAPACITORS:0603
- added L5, L6, L7, L8: 470uH, INDUCTORS:SRN1060
- added Q3: SI4848ADY, TRANSISTORs:SO8
- added R13: 10k, r_0603:0603
- added R14: 100R, RESISTORS:15MM_TH
- added R15: 240R, r_0603:0603
- added R16: 2.0k, r_0603:0603
- added U3: DCDC +/-15V, ICs:PDQE10
- added U4, U5: DCDC 15V, ICs:PDQE10
- added U6: LM317, ICs:TO220
Connections:
- removed net N$10: L3.2, L4.1
- new net AMP_12V: C16.2, C17.2, R15.2, U6.2
- new net DSP_AGND: C11.1, C12.2, U3.4
- new net DSP_DGND: C13.1, U4.5
- new net DSP_VA+: C11.2, L5.2
- new net DSP_VA-: C12.1, L6.2
- new net DSP_VD+: C13.2, L7.2
- new net N$12: L5.1, U3.3
- new net N$13: L6.1, U3.5
- new net N$14: R15.1, R16.2, U6.1
- new net N$18: C14.2, C15.2, L8.2, U6.3
- new net N$20: L8.1, U5.3
- new net N$22: L7.1, U4.3
- new net N$23: Q3.5, Q3.6, Q3.7, Q3.8, R14.1
- new net PGND: C14.1, C15.1, C16.1, C17.1, R16.1, U5.5
- net GND: now also Q3.1, Q3.2, Q3.3, R13.1, U3.1, U4.1, U5.1
- net N$4: now also L3.2, L4.1
- net PSU_VIN_OVERVOLT: now also Q3.4, R13.2
- net VIN: now also R14.2, U3.2, U4.2, U5.2

Commit message: Layout nearly complete
Parts:
- added C18: 100nF 16V, CAPACITORS:0603
- added HOLE1, HOLE2, HOLE3, HOLE4, HOLE5, HOLE6, HOLE7, HOLE8: 4mm ID, MISC:MOUNTHOLE_8X4
- added HOLE10, HOLE11, HOLE12, HOLE13, HOLE14, HOLE9: MOUNTHOLE_METAL4X2, MISC:4X2
- added MECH1, MECH2, MECH3, MECH4: 6mm x 3mm, MISC:MOUNTHOLE_6X3
- added R17: 100k, r_0603:0603
- R20: device r_0402:0402 -> r_0603:0603
- moved C17 676.3 mm to (51.2, 80.0)
- moved C16 661.2 mm to (50.0, 70.8), turned to 270 degrees
- moved C15 657.5 mm to (47.5, 70.8), turned to 270 degrees
- moved R16 655.9 mm to (52.0, 71.2)
- moved R15 651.5 mm to (52.0, 70.0), turned to 180 degrees
- moved U6 640.4 mm to (50.0, 66.5), turned to 180 degrees
- moved C12 638.8 mm to (47.5, 137.5), turned to 90 degrees
- moved C13 627.4 mm to (37.4, 105.0), turned to 180 degrees
- moved C14 616.0 mm to (37.4, 70.0), turned to 180 degrees
- moved C11 613.8 mm to (47.5, 122.5), turned to 90 degrees
- moved L7 596.3 mm to (35.0, 85.0)
- moved L6 592.4 mm to (35.0, 140.0)
- moved L8 584.9 mm to (35.0, 50.0)
- moved R14 581.1 mm to (55.0, 10.0), turned to 90 degrees
- moved R13 568.3 mm to (42.2, 4.25), turned to 270 degrees
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Connections:
- net 5V: now also C18.2
- net AMP_12V: now also HOLE10.1, HOLE12.1, HOLE14.1
- net GND: now also C18.1, HOLE2.1, HOLE3.1, HOLE5.1, HOLE7.1
- net N$1: now also C1.2, HOLE1.1
- net N$3: now also R17.2
- net N$8: now also R17.1; no longer C1.2
- net PGND: now also HOLE11.1, HOLE13.1, HOLE9.1
- net VOUT: now also HOLE4.1, HOLE6.1, HOLE8.1
Routing:
- net PGND: track 0.00 -> 327.6 mm, vias 0 -> 3
- net AMP_12V: track 0.00 -> 283.0 mm
- net VIN: track 0.00 -> 128.4 mm
- net DSP_VD+: track 0.00 -> 70.9 mm
- net DSP_DGND: track 0.00 -> 62.3 mm
- net PSU_VIN_OVERVOLT: track 0.00 -> 53.4 mm
- net DSP_AGND: track 0.00 -> 53.3 mm
- net DSP_VA+: track 0.00 -> 38.3 mm
- net N$8: track 0.00 -> 37.8 mm
- net GND: track 0.00 -> 32.0 mm, vias 0 -> 19
- net N$18: track 0.00 -> 31.1 mm
- net 5V: track 0.00 -> 29.7 mm
- net N$7: track 0.00 -> 25.4 mm
- net DSP_VA-: track 0.00 -> 16.3 mm
- net N$11: track 0.00 -> 15.1 mm
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- added copper zone on layer 1, net GND
- added copper zone on layer 16, net GND
- added copper zone on layer 1, net N$1
- added copper zone on layer 1, net N$4
- added copper zone on layer 1, net N$8
- added copper zone on layer 1, net VIN
- added copper zone on layer 1, net VOUT
Other:
- outline, holes or cut-outs redrawn
