File: sa_dsp.sch (EAGLE design)
At the start: 2 parts, among them U1 10CL016YF484C6G, U2 OSD3358-512M-BSM

Commit message: Work on the DSP
Parts:
- removed U2: OSD3358-512M-BSM, Octavo-Systems:OSD3358-512M-BSM
- added C10, C13, C14, C17, C2, C25, C26, C28, C3, C30, C35, C36, C37, C38, C43, C44, C47, C49, C5, C58, C59, C6, C60, C61, C62, C63, C64, C65, C66, C69, C71, C79, C8, C80, C81, C82, C83, C84, C9: 100nF 16V, CAPACITORS:CL10B104KO8WPNC
- added C11, C12, C16, C22, C45, C46, C48, C54, C67, C68, C7, C70, C76: 10uF 10V, CAPACITORS:GRM188R61A106KE69D
- added C15, C27: 15pF 50V, CAPACITORS:06035A150JAT2A
- added C18, C19, C20, C21, C50, C51, C52, C53, C72, C73, C74, C75: 470pF 16V, CAPACITORS:ECHU1C471GX5
- added C23, C24, C56, C57, C77, C78: 330nF 16V, CAPACITORS:ECPU1C334MA5
- added CN1: uSD, CONNECTORs:114-00841-68
- added D1, D2, D3, D4: RED STATUS, OPTO:VLMT3100-GS08
- added FB10, FB11, FB12, FB13, FB14, FB15, FB16, FB2, FB5, FB7, FB8, FB9: 600R, INDUCTORS:742792651
- added Q3, Q4: 2N7002, TRANSISTORs:2N7002P,215
- added R10, R11, R27, R28, R38, R39: 180k, r_0603:ERJ3EKF1803V
- added R108, R109, R110, R111, R112, R113, R114, R115, R18, R19, R45, R46, R47, R48, R49, R50, R51, R52, R6, R78, R79, R80, R82, R83, R92, R93, R94, R95, R96, R97, R98, R99: 470R, r_0603:ERJ3EKF4700V
- added R16, R17, R20, R21, R29, R30, R31, R32, R40, R41, R42, R43, R75, R76, R77, R81: 1.0k, r_0603:ERJ3EKF1001V
- added R2, R23, R24, R25, R26, R34, R35, R36, R37, R7, R8, R9: 20k, r_0603:ERJ3EKF2002V
- added R22, R33, R44: 22R, RESISTORS:EXB-38V220JV
- added R53: 10k, r_0603:ERJ3EKF1002V
- added R54, R55, R56, R57, R58, R59, R60, R61, R62, R63, R64, R65, R66, R67, R68, R69: 100k, r_0603:ERJ3EKF1003V
- added R70, R71: 10k, RESISTORS:EXB-38V103JV
- added R72, R73, R74: 1.0M, r_0603:ERJ3EKF1004V
- added U10, U12, U13, U15, U17, U18, U20, U4, U5: LME49720, ICs:LME49720MA/NOPB
- added U11, U16: PGA2311, ICs:PGA2311UA
- added U14, U19, U9: PCM1754, ICs:PCM1754
- added U21, U25, U29, U7: 7 SEG, OPTO:SC56-11SRWA
- added U22, U26, U30, U8: 74HC164A, ICs:MC74HC164ADTR2G
- added U3: OSD3358-512M-BSM, Octavo-Systems:OSD3358-512M-BSM
- added XTAL2: 24MHz, CRYSTALS:7A-24.000MAAJ-T
- U1: value 10CL016YF484C6G -> PGA2311; device ICs:10CL016YF484C6G -> ICs:PGA2311UA
Connections:
- new net +5V: C25.2, C28.2, C36.2, C58.2, C60.2, C62.2, C79.2, C81.2, C83.2, FB10.1, FB12.2, FB14.1, FB16.2, FB5.1, FB8.2, U10A.V+, U12A.V+, U13A.V+, U15A.V+, U17A.V+, U18A.V+, U20A.V+, U4A.V+, U5A.V+
- new net -5V: C26.1, C35.1, C37.1, C59.1, C61.1, C63.1, C80.1, C82.1, C84.1, FB13.1, FB2.1, FB9.1, U10A.V-, U12A.V-, U13A.V-, U15A.V-, U17A.V-, U18A.V-, U20A.V-, U4A.V-, U5A.V-
- new net 3V3: C2.2, C3.2, C30.2, C5.2, C6.2, C7.2, CN1.VCC, R54.2, R55.2, R56.2, R70.5, R70.6, R70.7, R70.8, R71.6, R71.7, R71.8, R72.2, U22.!RESET, U22.VCC, U26.!RESET, U26.VCC, U30.!RESET, U30.VCC, U8.!RESET, U8.VCC
- new net 5V: FB11.2, FB15.2, FB7.2, U1.ZCEN, U11.ZCEN, U16.ZCEN, U3A.VIN_AC@1, U3A.VIN_AC@2, U3A.VIN_AC@3, U3B.USB1_VBUS
- new net 5VUSB: U3B.USB0_VBUS
- new net AGND: C11.1, C12.1, C13.1, C16.1, C17.1, C18.2, C20.2, C22.1, C25.1, C26.2, C28.1, C35.2, C36.1, C37.2, C38.1, C43.1, C45.1, C46.1, C47.1, C48.1, C49.1, C50.2, C52.2, C54.1, C58.1, C59.2, C60.1, C61.2, C62.1, C63.2, C64.1, C65.1, C67.1, C68.1, C69.1, C70.1, C71.1, C72.2, C74.2, C76.1, C79.1, C8.1, C80.2, C81.1, C82.2, C83.1, C84.2, C9.1, R10.1, R11.1, R27.1, R28.1, R38.1, R39.1, U1.AGNDL, U1.AGNDR, U11.AGNDL, U11.AGNDR, U12B.+, U13B.+, U14.AGND, U16.AGNDL, U16.AGNDR, U17B.+, U18B.+, U19.AGND, U4B.+, U5B.+, U9.AGND
- new net AM_DEBUG_UART_RX: U3C.UART0_RXD
- new net AM_DEBUG_UART_TX: U3C.UART0_TXD
- new net AM_EEPROM_WP: U3A.EEPROM_WP, U3C.GPMC_BEN0_CLE
- new net AM_PMIC_PGOOD: Q4.G, R73.2, U3A.PMIC_PGOOD, U3A.PWRONRSTN
- new net AM_PWR_BTN: U3A.PMIC_PB_IN
- new net AM_STM_NRST: U3C.GPMC_AD9
- new net AM_USR_LED0: R75.1, U3C.GPMC_A5
- new net AM_USR_LED1: R76.1, U3C.GPMC_A6
- new net AM_USR_LED2: R77.1, U3C.GPMC_A7
- new net AM_USR_LED3: R81.1, U3C.GPMC_A8
- new net AM_WARM_!RST: Q3.D, U3A.WARMRSTN
- new net DAC0_I2S_BCLK: R22.8, R33.8, R44.8
- new net DAC0_I2S_DATA: R22.7, R33.7, R44.7
- new net DAC0_I2S_LRCLK: R22.6, R33.6, R44.6
- new net DAC0_I2S_SCLK: R22.5, R33.5, R44.5
- new net DAC_MUTE: U14.MUTE, U19.MUTE, U9.MUTE
- new net DISP_SPI_!CE: U22.A2, U26.A2, U30.A2, U8.A2
- new net DISP_SPI_MOSI: U22.A1, U26.A1, U30.A1, U8.A1
- new net DISP_SPI_SCLK: U22.CLK, U26.CLK, U30.CLK, U8.CLK
- new net GND: C10.1, C2.1, C3.1, C30.1, C44.1, C5.1, C6.1, C66.1, C7.1, CN1.C_D2, CN1.GND, D1.K, D2.K, D3.K, D4.K, Q3.S, Q4.S, R53.1, R57.1, R58.1, R59.1, R60.1, R61.1, R62.1, R63.1, R64.1, R65.1, R66.1, R67.1, R68.1, R69.1, R73.1, U1.DGND, U11.DGND, U14.DEMP, U14.DGND, U14.FMT, U14.TEST, U16.DGND, U19.DEMP, U19.DGND, U19.FMT, U19.TEST, U21.K, U22.GND, U25.K, U26.GND, U29.K, U30.GND, U3B.USB1_ID, U3E.DGND@1, U3E.DGND@10, U3E.DGND@11, U3E.DGND@12, U3E.DGND@13, U3E.DGND@14, U3E.DGND@15, U3E.DGND@16, U3E.DGND@17, U3E.DGND@18, U3E.DGND@19, U3E.DGND@2, U3E.DGND@20, U3E.DGND@21, U3E.DGND@22, U3E.DGND@23, U3E.DGND@24, U3E.DGND@25, U3E.DGND@26, U3E.DGND@27, U3E.DGND@28, U3E.DGND@29, U3E.DGND@3, U3E.DGND@30, U3E.DGND@31, U3E.DGND@32, U3E.DGND@33, U3E.DGND@34, U3E.DGND@35, U3E.DGND@36, U3E.DGND@4, U3E.DGND@5, U3E.DGND@6, U3E.DGND@7, U3E.DGND@8, U3E.DGND@9, U7.K, U8.GND, U9.DEMP, U9.DGND, U9.FMT, U9.TEST
- new net MMC0_CD: CN1.C_D1, R71.3, U3C.SPI0_CS1
- new net MMC0_CLK: CN1.CLK, R70.3, U3C.MMC0_CLK
- new net MMC0_CMD: CN1.C/R, R70.4, U3C.MMC0_CMD
- new net MMC0_D0: CN1.D0, R70.2, U3C.MMC0_DAT0
- new net MMC0_D1: CN1.D1, R70.1, U3C.MMC0_DAT1
- new net MMC0_D2: CN1.D2, R71.2, U3C.MMC0_DAT2
- new net MMC0_D3: CN1.D3, R71.1, U3C.MMC0_DAT3
- new net N$100: R41.2, U17B.OUT
- new net N$101: C78.2, R36.1, R39.2
- new net N$102: C77.2, R34.1, R38.2
- new net N$103: R44.1, U19.BCK
- new net N$104: R44.2, U19.DATA
- new net N$105: R44.4, U19.SCK
- new net N$106: R44.3, U19.LRCLK
- new net N$107: C77.1, U19.VOUT_R
- new net N$108: R40.1, U16.VOUTL, U17A.+
- new net N$109: R19.1, U8.QG
- new net N$11: C10.2, FB7.1, U1.VD+
- new net N$110: R6.1, U8.QF
- new net N$111: R18.1, U8.QE
- new net N$112: R50.2, U21.A
- new net N$113: R51.2, U21.B
- new net N$114: R52.2, U21.C
- new net N$115: R78.2, U21.D
- new net N$116: R79.1, U21.DP
- new net N$117: R80.1, U21.G
- new net N$118: R82.1, U21.F
- new net N$119: R83.1, U21.E
- new net N$12: U4A.-, U4A.OUT
- new net N$120: R80.2, U22.QD
- new net N$121: R82.2, U22.QC
- new net N$122: R83.2, U22.QA
- new net N$123: R78.1, U22.QB
- new net N$124: U3A.SYS_VOUT@1, U3A.SYS_VOUT@2, U3A.SYS_VOUT@3, U3A.SYS_VOUT@4
- new net N$125: U3A.SYS_VDD1_3P3V@1, U3A.SYS_VDD1_3P3V@2, U3A.SYS_VDD1_3P3V@3, U3A.SYS_VDD1_3P3V@4
- new net N$126: U3A.SYS_VDD2_3P3V@1, U3A.SYS_VDD2_3P3V@2
- new net N$127: U3A.SYS_RTC_1P8V@1, U3A.SYS_RTC_1P8V@2
- new net N$128: U3A.SYS_VDD3_3P3V@1, U3A.SYS_VDD3_3P3V@2, U3A.SYS_VDD3_3P3V@3, U3A.SYS_VDD3_3P3V@4, U3A.SYS_VDD3_3P3V@5, U3A.SYS_VDD3_3P3V@6, U3A.SYS_VDD3_3P3V@7, U3A.SYS_VDD3_3P3V@8, U3A.VDDSHV1, U3A.VDDSHV2, U3A.VDDSHV3, U3A.VDDSHV4, U3A.VDDSHV5, U3A.VDDSHV6
- new net N$129: U3A.SYS_VDD_1P8V@1, U3A.SYS_VDD_1P8V@2, U3A.SYS_VDD_1P8V@3, U3A.SYS_VDD_1P8V@4, U3A.SYS_VDD_1P8V@5, U3A.SYS_VDD_1P8V@6, U3A.SYS_VDD_1P8V@7, U3A.SYS_VDD_1P8V@8
- new net N$13: R16.2, R17.1, U4B.-
- new net N$130: U3A.PMIC_POWER_EN, U3A.PMIC_PWR_EN
- new net N$131: U3A.PMIC_LDO_PGOOD, U3A.RTC_PWRONRSTN
- new net N$132: U3A.EXT_WAKEUP, U3A.PMIC_NWAKEUP
- new net N$133: U3A.EXTINTN, U3A.PMIC_NINT
- new net N$134: U3A.I2C0_SCL, U3A.PMIC_SCL
- new net N$135: U3A.I2C0_SDA, U3A.PMIC_SDA
- new net N$136: R53.2, U3A.RTC_KALDO_ENN
- new net N$137: R57.2, U3D.LCD_DATA0
- new net N$138: R58.2, U3D.LCD_DATA1
- new net N$139: R59.2, U3D.LCD_DATA2
- new net N$140: R54.1, U3D.LCD_DATA3
- new net N$141: R55.1, U3D.LCD_DATA4
- new net N$142: R60.2, U3D.LCD_DATA5
- new net N$143: R61.2, U3D.LCD_DATA6
- new net N$144: R62.2, U3D.LCD_DATA7
- new net N$145: R63.2, U3D.LCD_DATA8
- new net N$146: R64.2, U3D.LCD_DATA9
- new net N$147: R65.2, U3D.LCD_DATA10
- new net N$148: R66.2, U3D.LCD_DATA11
- new net N$149: R67.2, U3D.LCD_DATA12
- new net N$150: R68.2, U3D.LCD_DATA13
- new net N$151: R56.1, U3D.LCD_DATA14
- new net N$152: R69.2, U3D.LCD_DATA15
- new net N$153: U3A.VIN_USB@1, U3A.VIN_USB@2, U3A.VIN_USB@3
- new net N$154: U3A.PMIC_BAT_SENSE, U3A.VIN_BAT@1, U3A.VIN_BAT@2, U3A.VIN_BAT@3
- new net N$155: C14.2, U3B.SYS_ADC_1P8V, U3B.VREFP
- new net N$156: C14.1, U3B.AGND_ADC, U3B.VREFN
- new net N$157: Q3.G, Q4.D, R72.1
- new net N$158: C27.2, R74.1, U3B.OSC0_OUT, XTAL2.P$2
- new net N$159: C15.2, R74.2, U3B.OSC0_IN, XTAL2.P$1
- new net N$160: C15.1, C27.1, U3B.OSC0_GND
- new net N$161: U3B.AIN7, U3B.PMIC_MUX_OUT
- new net N$162: D1.A, R75.2
- new net N$163: D2.A, R76.2
- new net N$164: D3.A, R77.2
- new net N$165: D4.A, R81.2
- new net N$166: R52.1, U22.QG
- new net N$167: R50.1, U22.QF
- new net N$168: R51.1, U22.QE
- new net N$17: U5A.-, U5A.OUT
- new net N$184: R92.2, U25.A
- new net N$185: R93.2, U25.B
- new net N$186: R94.2, U25.C
- new net N$187: R95.2, U25.D
- new net N$188: R96.1, U25.DP
- new net N$189: R97.1, U25.G
- new net N$190: R98.1, U25.F
- new net N$191: R99.1, U25.E
- new net N$192: R97.2, U26.QD
- new net N$193: R98.2, U26.QC
- new net N$194: R99.2, U26.QA
- new net N$195: R95.1, U26.QB
- new net N$196: R94.1, U26.QG
- new net N$197: R92.1, U26.QF
- new net N$198: R93.1, U26.QE
- new net N$214: R108.2, U29.A
- new net N$215: R109.2, U29.B
- new net N$216: R110.2, U29.C
- new net N$217: R111.2, U29.D
- new net N$218: R112.1, U29.DP
- new net N$219: R113.1, U29.G
- new net N$22: R6.2, U7.A
- new net N$220: R114.1, U29.F
- new net N$221: R115.1, U29.E
- new net N$222: R113.2, U30.QD
- new net N$223: R114.2, U30.QC
- new net N$224: R115.2, U30.QA
- new net N$225: R111.1, U30.QB
- new net N$226: R110.1, U30.QG
- new net N$227: R108.1, U30.QF
- new net N$228: R109.1, U30.QE
- new net N$23: R18.2, U7.B
- new net N$24: R19.2, U7.C
- new net N$25: R45.2, U7.D
- new net N$26: R20.1, U1.VOUTR, U5A.+
- new net N$27: R20.2, R21.1, U5B.-
- new net N$28: R21.2, U5B.OUT
- new net N$29: C13.2, C22.2, FB8.1, U9.VCC
- new net N$30: R46.1, U7.DP
- new net N$31: R47.1, U7.G
- new net N$32: R48.1, U7.F
- new net N$33: R49.1, U7.E
- new net N$34: C16.2, C17.2, U9.VCOM
- new net N$35: R47.2, U8.QD
- new net N$36: C19.2, R2.2, R7.1
- new net N$37: C18.1, R7.2, U10A.+
- new net N$38: R48.2, U8.QC
- new net N$39: R49.2, U8.QA
- new net N$40: C19.1, U1.VINR, U10A.-, U10A.OUT
- new net N$41: C21.2, R8.2, R9.1
- new net N$42: C20.1, R9.2, U10B.+
- new net N$43: R45.1, U8.QB
- new net N$44: C21.1, U1.VINL, U10B.-, U10B.OUT
- new net N$45: C24.1, U9.VOUT_L
- new net N$46: R17.2, U4B.OUT
- new net N$47: C24.2, R11.2, R8.1
- new net N$48: C23.2, R10.2, R2.1
- new net N$49: R22.1, U9.BCK
- new net N$50: R22.2, U9.DATA
- new net N$51: R22.4, U9.SCK
- new net N$52: R22.3, U9.LRCLK
- new net N$53: C23.1, U9.VOUT_R
- new net N$54: R16.1, U1.VOUTL, U4A.+
- new net N$55: C38.2, C45.2, FB9.2, U11.VA-
- new net N$56: C43.2, C46.2, FB10.2, U11.VA+
- new net N$57: C44.2, FB11.1, U11.VD+
- new net N$58: U12A.-, U12A.OUT
- new net N$59: R29.2, R30.1, U12B.-
- new net N$60: U13A.-, U13A.OUT
- new net N$61: R31.1, U11.VOUTR, U13A.+
- new net N$62: R31.2, R32.1, U13B.-
- new net N$63: R32.2, U13B.OUT
- new net N$64: C47.2, C54.2, FB12.1, U14.VCC
- new net N$65: C48.2, C49.2, U14.VCOM
- new net N$66: C51.2, R23.2, R24.1
- new net N$67: C50.1, R24.2, U15A.+
- new net N$68: C51.1, U11.VINR, U15A.-, U15A.OUT
- new net N$69: C53.2, R25.2, R26.1
- new net N$70: C52.1, R26.2, U15B.+
- new net N$71: C53.1, U11.VINL, U15B.-, U15B.OUT
- new net N$72: C57.1, U14.VOUT_L
- new net N$73: R30.2, U12B.OUT
- new net N$74: C57.2, R25.1, R28.2
- new net N$75: C56.2, R23.1, R27.2
- new net N$76: R33.1, U14.BCK
- new net N$77: R33.2, U14.DATA
- new net N$78: R33.4, U14.SCK
- new net N$79: R33.3, U14.LRCLK
- new net N$8: C11.2, C8.2, FB2.2, U1.VA-
- new net N$80: C56.1, U14.VOUT_R
- new net N$81: R29.1, U11.VOUTL, U12A.+
- new net N$82: C64.2, C67.2, FB13.2, U16.VA-
- new net N$83: C65.2, C68.2, FB14.2, U16.VA+
- new net N$84: C66.2, FB15.1, U16.VD+
- new net N$85: U17A.-, U17A.OUT
- new net N$86: R40.2, R41.1, U17B.-
- new net N$87: U18A.-, U18A.OUT
- new net N$88: R42.1, U16.VOUTR, U18A.+
- new net N$89: R42.2, R43.1, U18B.-
- new net N$9: C12.2, C9.2, FB5.2, U1.VA+
- new net N$90: R43.2, U18B.OUT
- new net N$91: C69.2, C76.2, FB16.1, U19.VCC
- new net N$92: C70.2, C71.2, U19.VCOM
- new net N$93: C73.2, R34.2, R35.1
- new net N$94: C72.1, R35.2, U20A.+
- new net N$95: C73.1, U16.VINR, U20A.-, U20A.OUT
- new net N$96: C75.2, R36.2, R37.1
- new net N$97: C74.1, R37.2, U20B.+
- new net N$98: C75.1, U16.VINL, U20B.-, U20B.OUT
- new net N$99: C78.1, U19.VOUT_L
- new net PGA0_!CS: U1.!CS, U11.!CS, U16.!CS
- new net PGA_!MUTE: U1.!MUTE, U11.!MUTE, U16.!MUTE
- new net PGA_SCLK: U1.SCLK, U11.SCLK, U16.SCLK
- new net PGA_SDI: U1.SDI, U11.SDI, U16.SDI
- new net SHIFT_OUT: R112.2, R46.2, R79.2, R96.2, U22.QH, U26.QH, U30.QH, U8.QH
- new net STM32_BOOT0: U3C.GPMC_AD10
- new net STM_AM_UART_RX: U3C.UART1_TXD
- new net STM_AM_UART_TX: U3C.UART1_RXD
- new net USB0_DM: U3B.USB0_DM
- new net USB0_DP: U3B.USB0_DP
- new net USB0_ID: U3B.USB0_ID
- new net USB1_DM: U3B.USB1_DM
- new net USB1_DP: U3B.USB1_DP

Commit message: Added FPGA
Parts:
- added C100, C101, C102, C103, C104, C105, C106, C107, C109, C110, C111, C112, C113, C114, C115, C116, C117, C118, C96, C97, C98, C99: 100nF 16V, CAPACITORS:CL05B104KO5NNNC
- added C108: 4.7uF 16V, CAPACITORS:CL05A475MO5NUNC
- added CN3: 2X5 HEADER, CONNECTORs:2X5_HEADER
- added MECH1, MECH2, MECH3, MECH4: 6mm x 3mm, MISC:MOUNTHOLE
- added R14: 1.0k, r_0603:ERJ3EKF1001V
- added R15, R84, R85, R86, R87: 10k, r_0603:ERJ3EKF1002V
- added U6: 10CL016YF484C6G, ICs:10CL016YF484C6G
Connections:
- new net 1V2: C100.2, C101.2, C102.2, C103.2, C104.2, C105.2, C106.2, C107.2, C108.2, U6.VCCD_PLL1, U6.VCCD_PLL2, U6.VCCD_PLL3, U6.VCCD_PLL4, U6.VCCINT
- new net 2V5: C96.2, C97.2, C98.2, C99.2, U6.VCCA1, U6.VCCA2, U6.VCCA3, U6.VCCA4
- new net CONF_CONFDN: R86.1, U6.B6_CONF_DONE
- new net CONF_JTAG_TCK: CN3.1, R14.2, U6.B1_TCK
- new net CONF_JTAG_TDI: CN3.5, R84.1, U6.B1_TDI
- new net CONF_JTAG_TDO: CN3.2, U6.B1_TDO
- new net CONF_JTAG_TMS: CN3.3, R15.1, U6.B1_TMS
- new net CONF_NCONFIG: R87.1
- new net CONF_NSTATUS: R85.1, U6.B1_NSTATUS
- net 3V3: now also C109.2, C110.2, C111.2, C112.2, C113.2, C114.2, C115.2, C116.2, C117.2, C118.2, CN3.9, R15.2, R84.2, R85.2, R86.2, R87.2, U6.B1_NCONFIG, U6.VCCIO1, U6.VCCIO2, U6.VCCIO3, U6.VCCIO4, U6.VCCIO5, U6.VCCIO6, U6.VCCIO7, U6.VCCIO8
- net GND: now also C100.1, C101.1, C102.1, C103.1, C104.1, C105.1, C106.1, C107.1, C108.1, C109.1, C110.1, C111.1, C112.1, C113.1, C114.1, C115.1, C116.1, C117.1, C118.1, C96.1, C97.1, C98.1, C99.1, CN3.10, CN3.6, R14.1, U6.B1_IO28, U6.B1_IO29, U6.B1_NCE, U6.B6_MSEL0, U6.B6_MSEL1, U6.B6_MSEL2, U6.B6_MSEL3, U6.GND, U6.GNDA1, U6.GNDA2, U6.GNDA3, U6.GNDA4

Commit message: USB added
Parts:
- added C42, C55, C85, C86, C92: 100nF 16V, CAPACITORS:CL10B104KO8WPNC
- added C87, C88, C91: 10uF 10V, CAPACITORS:GRM188R61A106KE69D
- added C89, C90: 10pF 100V, CAPACITORS:06031A100FAT2A
- added R100, R91: 1.5k, r_0603:ERJ3EKF1501V
- added R101: 1.0M, r_0603:ERJ3EKF1004V
- added R88, R89: 22R, r_0603:ERJ3EKF22R0V
- added R90: 10k, r_0603:ERJ3EKF1002V
- added U23: PCM2707, ICs:PCM2707PJT
- added XTAL3: 12MHz, CRYSTALS:ABM8-12.000MHZ-B2-T
Connections:
- removed net 5VUSB: U3B.USB0_VBUS
- removed net USB0_DM: U3B.USB0_DM
- removed net USB0_DP: U3B.USB0_DP
- removed net USB0_ID: U3B.USB0_ID
- removed net USB1_DM: U3B.USB1_DM
- removed net USB1_DP: U3B.USB1_DP
- new net N$14: C89.2, R101.1, U23.XTI, XTAL3.P$2
- new net N$15: C90.2, R101.2, U23.XTO, XTAL3.P$1
- new net N$16: R88.2, R91.1, U23.D+
- new net N$169: R100.1, U23.DT
- new net N$18: R89.2, U23.D-
- new net N$21: C91.2, U23.VCOM
- new net OSD_USB1_DM: R89.1, U3B.USB1_DM
- new net OSD_USB1_DP: R88.1, U3B.USB1_DP
- new net PCM_I2S_BCLK: U23.FUNC1
- new net PCM_I2S_DOUT: U23.DOUT
- new net PCM_I2S_LRCLK: U23.FUNC0
- new net PCM_I2S_MCLK: U23.FUNC2
- net 3V3: now also C42.2, C55.2, C85.2, C86.2, C87.2, C88.2, C92.2, R100.2, U23.TEST, U23.VBUS, U23.VCCL, U23.VCCP, U23.VCCR, U23.VDD
- net 5V: now also R90.2, R91.2, U23.HOST
- net GND: now also C42.1, C55.1, C85.1, C86.1, C87.1, C88.1, C89.1, C90.1, C91.1, C92.1, R90.1, U23.AGNDL, U23.AGNDR, U23.DGND, U23.FSEL, U23.FUNC3, U23.PGND, U23.PSEL, U23.ZGND, XTAL3.GND

Commit message: Additions
Parts:
- added C1, C119, C125, C29, C4, C93, C94, C95: 100nF 16V, CAPACITORS:CL10B104KO8WPNC
- added C120, C121, C124: 10uF 10V, CAPACITORS:GRM188R61A106KE69D
- added C122, C123: 10pF 100V, CAPACITORS:06031A100FAT2A
- added R1, R104, R12, R3: 10k, r_0603:ERJ3EKF1002V
- added R102, R103: 22R, r_0603:ERJ3EKF22R0V
- added R105, R106: 1.5k, r_0603:ERJ3EKF1501V
- added R107: 1.0M, r_0603:ERJ3EKF1004V
- added R13, R4, R5: 1.0k, r_0603:ERJ3EKF1001V
- added RE1: PEC11, ELECTROMECH:PEC11R-4225F-S0024
- added U24: PCM2707, ICs:PCM2707PJT
- added XTAL4: 12MHz, CRYSTALS:ABM8-12.000MHZ-B2-T
Connections:
- net PCM_I2S_BCLK renamed PCM_I2S_BCLK_BB
- net PCM_I2S_DOUT renamed PCM_I2S_DOUT_BB
- net PCM_I2S_LRCLK renamed PCM_I2S_LRCLK_BB
- net PCM_I2S_MCLK renamed PCM_I2S_MCLK_BB
- new net 5VUSB: R104.2, R105.2, U24.HOST
- new net ENC_A: C1.2, R4.2
- new net ENC_B: C4.2, R5.2
- new net ENC_SW: C29.2, R13.1
- new net N$1: R1.1, R4.1, RE1.A
- new net N$170: R102.2, R105.1, U24.D+
- new net N$171: R103.2, U24.D-
- new net N$172: R102.1
- new net N$173: R103.1
- new net N$174: C124.2, U24.VCOM
- new net N$175: R106.1, U24.DT
- new net N$19: C122.2, R107.1, U24.XTI, XTAL4.P$2
- new net N$2: R3.1, R5.1, RE1.B
- new net N$20: C123.2, R107.2, U24.XTO, XTAL4.P$1
- new net N$5: R12.1, R13.2, RE1.SW_A
- new net PCM_I2S_BCLK_EXT: U24.FUNC1
- new net PCM_I2S_DOUT_EXT: U24.DOUT
- new net PCM_I2S_LRCLK_EXT: U24.FUNC0
- new net PCM_I2S_MCLK_EXT: U24.FUNC2
- net 3V3: now also C119.2, C120.2, C121.2, C125.2, C93.2, C94.2, C95.2, R1.2, R106.2, R12.2, R3.2, U24.TEST, U24.VBUS, U24.VCCL, U24.VCCP, U24.VCCR, U24.VDD
- net GND: now also C1.1, C119.1, C120.1, C121.1, C122.1, C123.1, C124.1, C125.1, C29.1, C4.1, C93.1, C94.1, C95.1, R104.1, RE1.GND, RE1.SW_B, U24.AGNDL, U24.AGNDR, U24.DGND, U24.FSEL, U24.FUNC3, U24.PGND, U24.PSEL, U24.ZGND, XTAL4.GND
Other:
- moved on the sheet: C42, C55, C85, C86, C87, C88, C89, C90, C91, C92, R100, R101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

Commit message: Routing the DACs to the FPGA
Connections:
- removed net DAC_MUTE: U14.MUTE, U19.MUTE, U9.MUTE
- removed net PGA_!MUTE: U1.!MUTE, U11.!MUTE, U16.!MUTE
- removed net PGA_SCLK: U1.SCLK, U11.SCLK, U16.SCLK
- removed net PGA_SDI: U1.SDI, U11.SDI, U16.SDI
- new net DAC0_MUTE: U19.MUTE
- new net DAC1_I2S_BCLK: R33.8
- new net DAC1_I2S_DATA: R33.7
- new net DAC1_I2S_LRCLK: R33.6
- new net DAC1_I2S_SCLK: R33.5
- new net DAC1_MUTE: U14.MUTE
- new net DAC2_I2S_BCLK: R22.8
- new net DAC2_I2S_DATA: R22.7
- new net DAC2_I2S_LRCLK: R22.6
- new net DAC2_I2S_SCLK: R22.5
- new net DAC2_MUTE: U9.MUTE
- new net PGA0_!MUTE: U16.!MUTE
- new net PGA0_SCLK: U16.SCLK
- new net PGA0_SDI: U16.SDI
- new net PGA1_!CS: U11.!CS
- new net PGA1_!MUTE: U11.!MUTE
- new net PGA1_SCLK: U11.SCLK
- new net PGA1_SDI: U11.SDI
- new net PGA2_!CS: U1.!CS
- new net PGA2_!MUTE: U1.!MUTE
- new net PGA2_SCLK: U1.SCLK
- new net PGA2_SDI: U1.SDI
- net DAC0_I2S_BCLK: no longer R22.8, R33.8
- net DAC0_I2S_DATA: no longer R22.7, R33.7
- net DAC0_I2S_LRCLK: no longer R22.6, R33.6
- net DAC0_I2S_SCLK: no longer R22.5, R33.5
- net PGA0_!CS: no longer U1.!CS, U11.!CS

Commit message: Routing the anallogue section
Connections:
- new net DISP_SPI_MOSI1: R46.2, U22.A1, U8.QH
- new net DISP_SPI_MOSI2: R79.2, U22.QH, U26.A1
- new net DISP_SPI_MOSI3: R96.2, U26.QH, U30.A1
- net DISP_SPI_MOSI: no longer U22.A1, U26.A1, U30.A1
- net SHIFT_OUT: no longer R46.2, R79.2, R96.2, U22.QH, U26.QH, U8.QH

Commit message: General progress
Parts:
- added C126, C129, C130, C33, C34, C40: 100uF 50V, CAPACITORS:107CKR050M
- added C127, C128, C31, C32, C39, C41: 10nF 50V, CAPACITORS:CL10B103KB8NCNC
- added C131, C132: 100nF 16V, CAPACITORS:CL10B104KO8WPNC
- added D5, D6: RED STATUS, OPTO:VLMT3100-GS08
- added FB1, FB3, FB4: 600R, INDUCTORS:742792651
- added L1, L2, L3: 47uH 0.9A, INDUCTORS:SRN5040-470M
- added R116, R119, R120: 240R, r_0603:ERJ3EKF2400V
- added R117, R118, R121: 750R, r_0603:ERJ3EKF7500V
- added R122: 10k, r_0603:ERJ3EKF1002V
- added R123, R124, R125: 1.0k, r_0603:ERJ3EKF1001V
- added SW1: 1825910-7, ELECTROMECH:1825910-7
- added TP1, TP2: TEST_POINT_SQUARE, MISC:TEST_POINT_SQUARE
- added U2, U28: LM317, ICs:LM317T
- added U27: LM337, ICs:LM337SP
- added U31: 100MHz, CRYSTALS:510BBA100M000BAG
- CN3: value 2X5 HEADER -> 2X5_HEADER
- U23, U24: value PCM2707 -> PCM2707PJT
- XTAL3, XTAL4: value 12MHz -> ABM8-12.000MHZ-B2-T
Connections:
- new net 15VA+_UNREG: L1.1
- new net 15VA-_UNREG: L2.1
- new net 15VD_UNREG: L3.1
- new net 5VD: R90.2, R91.2, U23.HOST, U3A.VIN_AC@1, U3A.VIN_AC@2, U3A.VIN_AC@3, U3B.USB1_VBUS
- new net CLK_100M: U31.OUT, U6.B8_CLK10
- new net CLK_100M_OE: U31.!ST, U6.B8_IO5
- new net N$10: FB1.1, L1.2
- new net N$176: R120.1, R121.2, U28.ADJ
- new net N$177: R118.1, R119.2, U27.ADJ
- new net N$178: C127.2, C129.A, FB4.2, U28.VIN
- new net N$179: FB4.1, L3.2
- new net N$180: R122.1, R123.1, SW1.1
- new net N$181: D5.A, R124.2
- new net N$182: D6.A, R125.2
- new net N$3: R116.1, R117.2, U2.ADJ
- new net N$4: C39.1, C40.K, FB3.2, U27.VIN
- new net N$6: C31.2, C33.A, FB1.2, U2.VIN
- new net N$7: FB3.1, L2.2
- new net UI_INPUT_AIRPLAY: R124.1
- new net UI_INPUT_SEL: C132.2, R123.2
- new net UI_INPUT_USB: R125.1
- net +5V: now also C32.2, C34.A, R116.2, U2.VOUT
- net -5V: now also C126.K, C41.1, R119.1, U27.VOUT
- net 3V3: now also C131.2, R122.2, U31.VCC
- net 5V: now also C128.2, C130.A, R120.2, U28.VOUT; no longer R90.2, R91.2, U23.HOST, U3A.VIN_AC@1, U3A.VIN_AC@2, U3A.VIN_AC@3, U3B.USB1_VBUS
- net AGND: now also C126.A, C31.1, C32.1, C33.K, C34.K, C39.2, C40.A, C41.2, R117.1, R118.2, TP2.P$1
- net GND: now also C127.1, C128.1, C129.K, C130.K, C131.1, C132.1, D5.K, D6.K, R121.1, SW1.2, TP1.P$1, U31.GND

Commit message: Libraies sorted
Parts:
- CN3: value 2X5_HEADER -> 2X5 HEADER
- U23, U24: value PCM2707PJT -> PCM2707
- XTAL3, XTAL4: value ABM8-12.000MHZ-B2-T -> 12MHz
