File: sa_dsp.sch (EAGLE design)
At the start: 434 parts, among them CN1 uSD, CN2 MINI B USB, CN3 2X5 HEADER, CN4 MINI B USB, CN5 USB A, CN6 MINI B USB, Q1 2N7002, Q2 2N7002, Q3 2N7002, Q4 2N7002, SW1 1825910-7, U1 PGA2311, U10 LME49720, U11 PGA2311, U12 LME49720, U13 LME49720, U14 PCM1754, U15 LME49720, U16 PGA2311, U17 LME49720, U18 LME49720, U19 PCM1754, U2 LM317, U20 LME49720, U21 7 SEG, U22 74HC164A, U23 PCM2707, U24 PCM2707, U25 7 SEG, U26 74HC164A, U27 LM337, U28 LM317, U29 7 SEG, U3 OSD3358-512M-BSM, U30 74HC164A, U31 100MHz, U32 USBLC6-2SC6, U33 FT230X, U34 USBLC6-2SC6, U35 USBLC6-2SC6, U36 USBLC6-2SC6, U37 2 PORT HUB, U38 TPS70925, U39 LM22670, U4 LME49720, U40 MPM3820, U41 MPM3820, U42 SN74LVC1G17D, U43 SN74LVC1G17D, U44 SN74LVC1G17D, U45 SN74LVC1G17D, U5 LME49720, U6 10CL016YF484C6G, U7 7 SEG, U8 74HC164A, U9 PCM1754

Commit message: amp fixed
Parts:
- removed C10, C119, C125, C13, C131, C132, C135, C136, C137, C139, C14, C141, C151, C152, C153, C154, C155, C156, C161, C162, C163, C164, C17, C2, C25, C26, C28, C29, C3, C30, C35, C36, C37, C38, C4, C42, C43, C44, C47, C49, C5, C55, C58, C59, C6, C60, C61, C62, C63, C64, C65, C66, C69, C71, C79, C8, C80, C81, C82, C83, C84, C85, C86, C9, C92, C93, C94, C95: 100nF 16V, CAPACITORS:CL10B104KO8WPNC
- removed C100, C101, C102, C103, C104, C105, C106, C107, C109, C110, C111, C112, C113, C114, C115, C116, C117, C118, C96, C97, C98, C99: 100nF 16V, CAPACITORS:CL05B104KO5NNNC
- removed C108: 4.7uF 16V, CAPACITORS:CL05A475MO5NUNC
- removed C11, C12, C120, C121, C124, C16, C22, C45, C46, C48, C54, C67, C68, C7, C70, C76, C87, C88, C91: 10uF 10V, CAPACITORS:GRM188R61A106KE69D
- removed C122, C123, C149, C150, C89, C90: 10pF 100V, CAPACITORS:06031A100FAT2A
- removed C126, C129, C130, C33, C34, C40: 100uF 50V, CAPACITORS:107CKR050M
- removed C127, C128, C147, C31, C32, C39, C41: 10nF 50V, CAPACITORS:CL10B103KB8NCNC
- removed C133, C144: 2.2uF 25V, CAPACITORS:GRM188R61E225KA12D
- removed C134, C138, C140: 100pF 50V, CAPACITORS:C0603C101K5GACTU
- removed C142, C157: 47uF 25V, CAPACITORS:C3216X5R1E476M160AC
- removed C143: 1uF 25V, CAPACITORS:CL10A105KA8NNNC
- removed C145, C146, C159, C160: 22uF 10V, CAPACITORS:CL31B226MPHNNNE
- removed C148: 47uF 10V, CAPACITORS:GRM31CR61A476ME15L
- removed C15, C27: 15pF 50V, CAPACITORS:06035A150JAT2A
- removed C158: 100nF 100V, CAPACITORS:06031C104KAT2A
- removed C18, C19, C20, C21, C50, C51, C52, C53, C72, C73, C74, C75: 470pF 16V, CAPACITORS:ECHU1C471GX5
- removed C23, C24, C56, C57, C77, C78: 330nF 16V, CAPACITORS:ECPU1C334MA5
- removed D10, D7: CG0603MLC, DIODES:CG0603MLC-12LE
- removed D11, D9: B0540W, DIODES:B0540W
- removed D6: RED STATUS, OPTO:VLMT3100-GS08
- removed D8: BC560, DIODES:BC560C
- removed FB1, FB10, FB11, FB12, FB13, FB14, FB15, FB16, FB17, FB18, FB2, FB3, FB4, FB5, FB6, FB7, FB8, FB9: 600R, INDUCTORS:742792651
- removed L1, L2, L3: 47uH 0.9A, INDUCTORS:SRN5040-470M
- removed L5: 47uH 3.1A, INDUCTORS:SRR1210-470M
- removed Q1, Q2, Q3, Q4: 2N7002, TRANSISTORs:2N7002P,215
- removed R10, R11, R27, R28, R38, R39: 180k, r_0603:ERJ3EKF1803V
- removed R100, R105, R106, R91: 1.5k, r_0603:ERJ3EKF1501V
- removed R101, R107, R139, R72, R73, R74: 1.0M, r_0603:ERJ3EKF1004V
- removed R102, R103, R88, R89: 22R, r_0603:ERJ3EKF22R0V
- removed R104, R12, R122, R133, R15, R53, R84, R85, R86, R90: 10k, r_0603:ERJ3EKF1002V
- removed R108, R109, R110, R111, R112, R113, R114, R115, R18, R19, R45, R46, R47, R48, R49, R50, R51, R52, R6, R78, R79, R80, R82, R83, R92, R93, R94, R95, R96, R97, R98, R99: 470R, r_0603:ERJ3EKF4700V
- removed R116, R119, R120: 240R, r_0603:ERJ3EKF2400V
- removed R117, R118, R121: 750R, r_0603:ERJ3EKF7500V
- removed R123, R124, R125, R13, R14, R16, R17, R20, R21, R29, R30, R31, R32, R40, R41, R42, R43, R75, R76, R77, R81: 1.0k, r_0603:ERJ3EKF1001V
- removed R126, R127, R130: 22k, r_0603:ERJ3EKF2202V
- removed R128: 160k, r_0603:ERJ3EKF1603V
- removed R129, R131, R132, R54, R55, R56, R57, R58, R59, R60, R61, R62, R63, R64, R65, R66, R67, R68, R69: 100k, r_0603:ERJ3EKF1003V
- removed R134, R23, R24, R25, R26, R34, R35, R36, R37, R7, R8, R9: 20k, r_0603:ERJ3EKF2002V
- removed R135, R137, R138: 51k, r_0603:ERJ3EKF5102V
- removed R136: 12k, r_0603:ERJ3EKF1202V
- removed R22, R33, R44: 22R, RESISTORS:EXB-38V220JV
- removed R70, R71: 10k, RESISTORS:EXB-38V103JV
- removed RE1: PEC11, ELECTROMECH:PEC11R-4225F-S0024
- removed SW1: 1825910-7, ELECTROMECH:1825910-7
- removed TP1, TP10, TP11, TP12, TP2, TP8, TP9: TEST_POINT_SQUARE, MISC:TEST_POINT_SQUARE
- removed TP13, TP14, TP15, TP16, TP17, TP18, TP19, TP20, TP21, TP22, TP23, TP24, TP25, TP26, TP27, TP28, TP29, TP3, TP30, TP31, TP32, TP33, TP34, TP4, TP5, TP6, TP7: 2MM_TEST_POINT, MISC:2MM_TEST_POINT
- removed U10, U12, U13, U15, U17, U18, U20, U4, U5: LME49720, ICs:LME49720MA/NOPB
- removed U11, U16: PGA2311, ICs:PGA2311UA
- removed U14, U19, U9: PCM1754, ICs:PCM1754
- removed U21, U25, U29, U7: 7 SEG, OPTO:SC56-11SRWA
- removed U22, U26, U30, U8: 74HC164A, ICs:MC74HC164ADTR2G
- removed U23, U24: PCM2707, ICs:PCM2707PJT
- removed U27: LM337, ICs:LM337SP
- removed U28: LM317, ICs:LM317T
- removed U3: OSD3358-512M-BSM, Octavo-Systems:OSD3358-512M-BSM
- removed U31: 100MHz, CRYSTALS:510BBA100M000BAG
- removed U32, U34, U35, U36: USBLC6-2SC6, ICs:USBLC6-2SC6
- removed U33: FT230X, ICs:FT230XS
- removed U37: 2 PORT HUB, ICs:USB2412
- removed U38: TPS70925, ICs:TPS70925DBVR
- removed U39: LM22670, ICs:LM22670MRX-5.0/NOPB
- removed U40, U41: MPM3820, ICs:MPM3820GQV-Z
- removed U42, U43, U44, U45: SN74LVC1G17D, ICs:SN74LVC1G17DBVR
- removed U6: 10CL016YF484C6G, ICs:10CL016YF484C6G
- removed XTAL2, XTAL5: 24MHz, CRYSTALS:7A-24.000MAAJ-T
- removed XTAL3, XTAL4: 12MHz, CRYSTALS:ABM8-12.000MHZ-B2-T
- added MECH5, MECH6, MECH7, MECH8, MECH9: 6mm x 3mm, MISC:MOUNTHOLE
- added RPI-CM1: RPI-CM4, RPI-CM4:RPI-CM4
- C1: value 100nF 16V -> 0.1uF 50V; device CAPACITORS:CL10B104KO8WPNC -> c_0603:CL10B104KB8NNWC
- CN1: value uSD -> 2-1761465-1; device CONNECTORs:114-00841-68 -> CONNECTORs:2-1761465-1
- CN2: value MINI B USB -> USB A; device CONNECTORs:MUSB-05-S-B-SM-A -> CONNECTORs:629104190121
- CN3: value 2X5 HEADER -> Gb RJ45 + MAG; device CONNECTORs:2X5_HEADER -> CONNECTORs:0857931020
- CN4, CN6: value MINI B USB -> PCB Tab; device CONNECTORs:MUSB-05-S-B-SM-A -> CONNECTORs:PCB_TAB
- CN5: value USB A -> PCB Tab; device CONNECTORs:629104190121 -> CONNECTORs:PCB_TAB
- D1, D2, D3, D4, D5: value RED STATUS -> RED LED; device OPTO:VLMT3100-GS08 -> OPTO:150060RS75000
- R1, R3: value 10k -> 1k; device r_0603:ERJ3EKF1002V -> r_0603:CRCW06031K00FKEB
- R2: value 20k -> 1k; device r_0603:ERJ3EKF2002V -> r_0603:CRCW06031K00FKEB
- R4, R5: value 1.0k -> 1k; device r_0603:ERJ3EKF1001V -> r_0603:CRCW06031K00FKEB
- U1: value PGA2311 -> DCDC 3V3; device ICs:PGA2311UA -> ICs:PDQE15-Q24-S3-D
- U2: value LM317 -> USBLC6-2SC6; device ICs:LM317T -> ICs:USBLC6-2SC6
Connections:
- removed net +5V: C25.2, C28.2, C32.2, C34.A, C36.2, C58.2, C60.2, C62.2, C79.2, C81.2, C83.2, FB10.1, FB12.2, FB14.1, FB16.2, FB5.1, FB8.2, R116.2, U10A.V+, U12A.V+, U13A.V+, U15A.V+, U17A.V+, U18A.V+, U2.VOUT, U20A.V+, U4A.V+, U5A.V+
- removed net -5V: C126.K, C26.1, C35.1, C37.1, C41.1, C59.1, C61.1, C63.1, C80.1, C82.1, C84.1, FB13.1, FB2.1, FB9.1, R119.1, U10A.V-, U12A.V-, U13A.V-, U15A.V-, U17A.V-, U18A.V-, U20A.V-, U27.VOUT, U4A.V-, U5A.V-
- removed net 15VA+_UNREG: L1.1, TP10.P$1
- removed net 15VA-_UNREG: L2.1, TP12.P$1
- removed net 15VD_UNREG: C142.1, C157.1, C158.2, D11.K, D9.K, L3.1, TP13.P$1, TP15.P$1, TP8.P$1, U39.VIN
- removed net 1V2: C100.2, C101.2, C102.2, C103.2, C104.2, C105.2, C106.2, C107.2, C108.2, C146.2, R126.2, U40.OUT, U40.OUT_S, U6.VCCD_PLL1, U6.VCCD_PLL2, U6.VCCD_PLL3, U6.VCCD_PLL4, U6.VCCINT
- removed net 2V5: C144.2, C96.2, C97.2, C98.2, C99.2, U38.VOUT, U6.VCCA1, U6.VCCA2, U6.VCCA3, U6.VCCA4
- removed net 5VD: C140.2, C141.2, C143.2, C145.2, C148.2, C156.2, C159.2, FB18.2, L5.2, R90.2, R91.2, U23.HOST, U35.VBUS, U38.EN, U38.VIN, U39.FB, U3A.VIN_AC@1, U3A.VIN_AC@2, U3A.VIN_AC@3, U3B.USB0_VBUS, U40.EN, U40.VIN, U41.EN, U41.VIN
- removed net 5VUSB: C138.2, C139.2, FB17.2, R104.2, R105.2, U24.HOST, U34.VBUS
- removed net AGND: C11.1, C12.1, C126.A, C13.1, C16.1, C17.1, C18.2, C20.2, C22.1, C25.1, C26.2, C28.1, C31.1, C32.1, C33.K, C34.K, C35.2, C36.1, C37.2, C38.1, C39.2, C40.A, C41.2, C43.1, C45.1, C46.1, C47.1, C48.1, C49.1, C50.2, C52.2, C54.1, C58.1, C59.2, C60.1, C61.2, C62.1, C63.2, C64.1, C65.1, C67.1, C68.1, C69.1, C70.1, C71.1, C72.2, C74.2, C76.1, C79.1, C8.1, C80.2, C81.1, C82.2, C83.1, C84.2, C9.1, R10.1, R11.1, R117.1, R118.2, R27.1, R28.1, R38.1, R39.1, TP11.P$1, TP18.P$1, TP2.P$1, TP21.P$1, TP24.P$1, TP27.P$1, TP30.P$1, TP33.P$1, U1.AGNDL, U1.AGNDR, U11.AGNDL, U11.AGNDR, U12B.+, U13B.+, U14.AGND, U16.AGNDL, U16.AGNDR, U17B.+, U18B.+, U19.AGND, U4B.+, U5B.+, U9.AGND
- removed net AM_DEBUG_UART_RX: U33.RXD, U3C.UART0_RXD
- removed net AM_DEBUG_UART_TX: U33.TXD, U3C.UART0_TXD
- removed net AM_EEPROM_WP: TP5.P$1, U3A.EEPROM_WP, U3C.GPMC_BEN0_CLE
- removed net AM_I2C0_SCL: TP3.P$1, U3A.I2C0_SCL, U3A.PMIC_SCL
- removed net AM_I2C0_SDA: TP4.P$1, U3A.I2C0_SDA, U3A.PMIC_SDA
- removed net AM_PMIC_PGOOD: Q4.G, R73.2, U3A.PMIC_PGOOD, U3A.PWRONRSTN
- removed net AM_PWR_BTN: U3A.PMIC_PB_IN, U6.B2_IO14
- removed net AM_USR_LED0: R75.1, U3C.GPMC_A5
- removed net AM_USR_LED1: R76.1, U3C.GPMC_A6
- removed net AM_USR_LED2: R77.1, U3C.GPMC_A7
- removed net AM_USR_LED3: R81.1, U3C.GPMC_A8
- removed net AM_WARM_!RST: Q3.D, TP7.P$1, U3A.WARMRSTN
- removed net CLK_100M: U31.OUT, U6.B8_CLK10
- removed net CLK_100M_OE: U31.!ST, U6.B8_IO5
- removed net CONF_CONFDN: R86.1, U6.B6_CONF_DONE
- removed net CONF_JTAG_TCK: CN3.1, R14.2, U6.B1_TCK
- removed net CONF_JTAG_TDI: CN3.5, R84.1, U6.B1_TDI
- removed net CONF_JTAG_TDO: CN3.2, U6.B1_TDO
- removed net CONF_JTAG_TMS: CN3.3, R15.1, U6.B1_TMS
- removed net CONF_NSTATUS: R85.1, U6.B1_NSTATUS
- removed net DAC0_I2S_BCLK: R44.8, U6.B5_IO13
- removed net DAC0_I2S_DATA: R44.7, U6.B5_IO12
- removed net DAC0_I2S_LRCLK: R44.6, U6.B5_IO21
- removed net DAC0_I2S_SCLK: R44.5, U6.B5_IO20
- removed net DAC0_MUTE: U19.MUTE, U6.B5_IO24
- removed net DAC1_I2S_BCLK: R33.8, U6.B5_IO31
- removed net DAC1_I2S_DATA: R33.7, U6.B5_IO38
- removed net DAC1_I2S_LRCLK: R33.6, U6.B5_IO37
- removed net DAC1_I2S_SCLK: R33.5, U6.B5_IO40
- removed net DAC1_MUTE: U14.MUTE, U6.B5_IO39
- removed net DAC2_I2S_BCLK: R22.8, U6.B6_IO18
- removed net DAC2_I2S_DATA: R22.7, U6.B6_IO19
- removed net DAC2_I2S_LRCLK: R22.6, U6.B6_IO22
- removed net DAC2_I2S_SCLK: R22.5, U6.B6_IO23
- removed net DAC2_MUTE: U6.B6_IO27, U9.MUTE
- removed net DISP_SPI_!CE: U22.A2, U26.A2, U30.A2, U6.B8_IO29, U8.A2
- removed net DISP_SPI_MOSI: U6.B8_IO24, U8.A1
- removed net DISP_SPI_MOSI1: R46.2, U22.A1, U8.QH
- removed net DISP_SPI_MOSI2: R79.2, U22.QH, U26.A1
- removed net DISP_SPI_MOSI3: R96.2, U26.QH, U30.A1
- removed net DISP_SPI_SCLK: U22.CLK, U26.CLK, U30.CLK, U6.B8_IO15, U8.CLK
- removed net ENC_A: U42.Q, U6.B8_IO33
- removed net ENC_B: U43.Q, U6.B8_IO13
- removed net ENC_SW: U44.Q, U6.B8_IO30
- removed net FT_DB_3V3: C133.2, C137.2, U33.!CTS, U33.!RESET, U33.3V3OUT, U33.VCCIO
- removed net FT_DB_USB_5V: C134.2, C135.2, C136.2, FB6.2, U32.VBUS, U33.VCC
- removed net IO_AUDIO_RLY_EN: Q2.G, R132.2, U6.B2_IO20
- removed net MMC0_CD: CN1.C_D1, R71.3, U3C.SPI0_CS1
- removed net MMC0_CLK: CN1.CLK, R70.3, U3C.MMC0_CLK
- removed net MMC0_CMD: CN1.C/R, R70.4, U3C.MMC0_CMD
- removed net MMC0_D0: CN1.D0, R70.2, U3C.MMC0_DAT0
- removed net MMC0_D1: CN1.D1, R70.1, U3C.MMC0_DAT1
- removed net MMC0_D2: CN1.D2, R71.2, U3C.MMC0_DAT2
- removed net MMC0_D3: CN1.D3, R71.1, U3C.MMC0_DAT3
- removed net N$10: FB1.1, L1.2
- removed net N$100: R41.2, TP19.P$1, U17B.OUT
- removed net N$101: C78.2, R36.1, R39.2
- removed net N$102: C77.2, R34.1, R38.2
- removed net N$103: R44.1, U19.BCK
- removed net N$104: R44.2, U19.DATA
- removed net N$105: R44.4, U19.SCK
- removed net N$106: R44.3, U19.LRCLK
- removed net N$107: C77.1, U19.VOUT_R
- removed net N$108: R40.1, U16.VOUTL, U17A.+
- removed net N$109: R19.1, U8.QG
- removed net N$11: C10.2, FB7.1, U1.VD+
- removed net N$110: R6.1, U8.QF
- removed net N$111: R18.1, U8.QE
- removed net N$112: R50.2, U21.A
- removed net N$113: R51.2, U21.B
- removed net N$114: R52.2, U21.C
- removed net N$115: R78.2, U21.D
- removed net N$116: R79.1, U21.DP
- removed net N$117: R80.1, U21.G
- removed net N$118: R82.1, U21.F
- removed net N$119: R83.1, U21.E
- removed net N$12: TP29.P$1, U4A.-, U4A.OUT
- removed net N$120: R80.2, U22.QD
- removed net N$121: R82.2, U22.QC
- removed net N$122: R83.2, U22.QA
- removed net N$123: R78.1, U22.QB
- removed net N$124: U3A.SYS_VOUT@1, U3A.SYS_VOUT@2, U3A.SYS_VOUT@3, U3A.SYS_VOUT@4
- removed net N$125: U3A.SYS_VDD1_3P3V@1, U3A.SYS_VDD1_3P3V@2, U3A.SYS_VDD1_3P3V@3, U3A.SYS_VDD1_3P3V@4
- removed net N$126: U3A.SYS_VDD2_3P3V@1, U3A.SYS_VDD2_3P3V@2
- removed net N$127: U3A.SYS_RTC_1P8V@1, U3A.SYS_RTC_1P8V@2
- removed net N$128: U3A.SYS_VDD3_3P3V@1, U3A.SYS_VDD3_3P3V@2, U3A.SYS_VDD3_3P3V@3, U3A.SYS_VDD3_3P3V@4, U3A.SYS_VDD3_3P3V@5, U3A.SYS_VDD3_3P3V@6, U3A.SYS_VDD3_3P3V@7, U3A.SYS_VDD3_3P3V@8, U3A.VDDSHV1, U3A.VDDSHV2, U3A.VDDSHV3, U3A.VDDSHV4, U3A.VDDSHV5, U3A.VDDSHV6
- removed net N$129: U3A.SYS_VDD_1P8V@1, U3A.SYS_VDD_1P8V@2, U3A.SYS_VDD_1P8V@3, U3A.SYS_VDD_1P8V@4, U3A.SYS_VDD_1P8V@5, U3A.SYS_VDD_1P8V@6, U3A.SYS_VDD_1P8V@7, U3A.SYS_VDD_1P8V@8
- removed net N$13: R16.2, R17.1, U4B.-
- removed net N$130: U3A.PMIC_POWER_EN, U3A.PMIC_PWR_EN
- removed net N$131: U3A.PMIC_LDO_PGOOD, U3A.RTC_PWRONRSTN
- removed net N$132: U3A.EXT_WAKEUP, U3A.PMIC_NWAKEUP
- removed net N$133: U3A.EXTINTN, U3A.PMIC_NINT
- removed net N$134: CN4.D-, U34.D-OUT
- removed net N$135: CN4.D+, U34.D+_OUT
- removed net N$136: R53.2, U3A.RTC_KALDO_ENN
- removed net N$137: R57.2, U3D.LCD_DATA0
- removed net N$138: R58.2, U3D.LCD_DATA1
- removed net N$139: R59.2, U3D.LCD_DATA2
- removed net N$14: C89.2, R101.1, U23.XTI, XTAL3.P$2
- removed net N$140: R54.1, U3D.LCD_DATA3
- removed net N$141: R55.1, U3D.LCD_DATA4
- removed net N$142: R60.2, U3D.LCD_DATA5
- removed net N$143: R61.2, U3D.LCD_DATA6
- removed net N$144: R62.2, U3D.LCD_DATA7
- removed net N$145: R63.2, U3D.LCD_DATA8
- removed net N$146: R64.2, U3D.LCD_DATA9
- removed net N$147: R65.2, U3D.LCD_DATA10
- removed net N$148: R66.2, U3D.LCD_DATA11
- removed net N$149: R67.2, U3D.LCD_DATA12
- removed net N$15: C90.2, R101.2, U23.XTO, XTAL3.P$1
- removed net N$150: R68.2, U3D.LCD_DATA13
- removed net N$151: R56.1, U3D.LCD_DATA14
- removed net N$152: R69.2, U3D.LCD_DATA15
- removed net N$153: U3A.VIN_USB@1, U3A.VIN_USB@2, U3A.VIN_USB@3
- removed net N$154: U3A.PMIC_BAT_SENSE, U3A.VIN_BAT@1, U3A.VIN_BAT@2, U3A.VIN_BAT@3
- removed net N$155: C14.2, U3B.SYS_ADC_1P8V, U3B.VREFP
- removed net N$156: C14.1, U3B.AGND_ADC, U3B.VREFN
- removed net N$157: Q3.G, Q4.D, R72.1
- removed net N$158: C27.2, R74.1, U3B.OSC0_OUT, XTAL2.P$2
- removed net N$159: C15.2, R74.2, U3B.OSC0_IN, XTAL2.P$1
- removed net N$16: R88.2, R91.1, U23.D+
- removed net N$160: C15.1, C27.1, U3B.OSC0_GND
- removed net N$161: U3B.AIN7, U3B.PMIC_MUX_OUT
- removed net N$162: D1.A, R75.2
- removed net N$163: D2.A, R76.2
- removed net N$164: D3.A, R77.2
- removed net N$165: D4.A, R81.2
- removed net N$166: R52.1, U22.QG
- removed net N$167: R50.1, U22.QF
- removed net N$168: R51.1, U22.QE
- removed net N$169: R100.1, U23.DT
- removed net N$17: TP32.P$1, U5A.-, U5A.OUT
- removed net N$170: R102.2, R105.1, U24.D+
- removed net N$171: R103.2, U24.D-
- removed net N$172: R103.1, U34.D-_IN
- removed net N$173: R102.1, U34.D+_IN
- removed net N$174: C124.2, U24.VCOM
- removed net N$175: R106.1, U24.DT
- removed net N$176: R120.1, R121.2, U28.ADJ
- removed net N$177: R118.1, R119.2, U27.ADJ
- removed net N$178: C127.2, C129.A, FB4.2, U28.VIN
- removed net N$179: FB4.1, L3.2
- removed net N$18: R89.2, U23.D-
- removed net N$180: R122.1, R123.1, SW1.1
- removed net N$181: D5.A, R124.2
- removed net N$182: D6.A, R125.2
- removed net N$183: CN2.D-, U32.D+_OUT
- removed net N$184: R92.2, U25.A
- removed net N$185: R93.2, U25.B
- removed net N$186: R94.2, U25.C
- removed net N$187: R95.2, U25.D
- removed net N$188: R96.1, U25.DP
- removed net N$189: R97.1, U25.G
- removed net N$19: C122.2, R107.1, U24.XTI, XTAL4.P$2
- removed net N$190: R98.1, U25.F
- removed net N$191: R99.1, U25.E
- removed net N$192: R97.2, U26.QD
- removed net N$193: R98.2, U26.QC
- removed net N$194: R99.2, U26.QA
- removed net N$195: R95.1, U26.QB
- removed net N$196: R94.1, U26.QG
- removed net N$197: R92.1, U26.QF
- removed net N$198: R93.1, U26.QE
- removed net N$199: CN2.D+, U32.D-OUT
- removed net N$20: C123.2, R107.2, U24.XTO, XTAL4.P$1
- removed net N$200: U32.D+_IN, U33.D-
- removed net N$201: U32.D-_IN, U33.D+
- removed net N$202: CN2.5V, FB6.1
- removed net N$203: CN4.5V, FB17.1
- removed net N$204: CN5.D-, U35.D-OUT
- removed net N$205: CN5.D+, U35.D+_OUT
- removed net N$206: CN5.VBUS, FB18.1
- removed net N$207: D7.A1, D9.A, Q1.D, TP14.P$1
- removed net N$208: CN6.D+, U36.D+_OUT
- removed net N$209: CN6.D-, U36.D-OUT
- removed net N$21: C91.2, U23.VCOM
- removed net N$210: R126.1, R127.2, U40.FB
- removed net N$211: R129.1, R130.2, U41.FB
- removed net N$212: C147.1, U39.BOOT
- removed net N$213: C147.2, D8.K, L5.1, U39.SW
- removed net N$214: R108.2, U29.A
- removed net N$215: R109.2, U29.B
- removed net N$216: R110.2, U29.C
- removed net N$217: R111.2, U29.D
- removed net N$218: R112.1, U29.DP
- removed net N$219: R113.1, U29.G
- removed net N$22: R6.2, U7.A
- removed net N$220: R114.1, U29.F
- removed net N$221: R115.1, U29.E
- removed net N$222: R113.2, U30.QD
- removed net N$223: R114.2, U30.QC
- removed net N$224: R115.2, U30.QA
- removed net N$225: R111.1, U30.QB
- removed net N$226: R110.1, U30.QG
- removed net N$227: R108.1, U30.QF
- removed net N$228: R109.1, U30.QE
- removed net N$229: R133.2, R134.2, U37.VBUS_DECT
- removed net N$23: R18.2, U7.B
- removed net N$230: R135.2, U37.HS_IND
- removed net N$231: R136.2, U37.RBIAS
- removed net N$232: R138.2, U37.NON_REM1
- removed net N$233: R137.2, U37.SUSP_IND/NON_REM0
- removed net N$234: C150.2, R139.2, U37.XTALIN/CLKLIN, XTAL5.P$1
- removed net N$235: C149.2, R139.1, U37.XTALOUT, XTAL5.P$2
- removed net N$236: R128.2, U39.RT_SYNC
- removed net N$237: D10.A1, D11.A, Q2.D, TP16.P$1
- removed net N$238: C4.2, R5.2, U43.A
- removed net N$239: C1.2, R4.2, U42.A
- removed net N$24: R19.2, U7.C
- removed net N$240: C29.2, R13.1, U44.A
- removed net N$241: C132.2, R123.2, U45.A
- removed net N$25: R45.2, U7.D
- removed net N$26: R20.1, U1.VOUTR, U5A.+
- removed net N$27: R20.2, R21.1, U5B.-
- removed net N$28: R21.2, TP34.P$1, U5B.OUT
- removed net N$29: C13.2, C22.2, FB8.1, U9.VCC
- removed net N$30: R46.1, U7.DP
- removed net N$31: R47.1, U7.G
- removed net N$32: R48.1, U7.F
- removed net N$33: R49.1, U7.E
- removed net N$34: C16.2, C17.2, U9.VCOM
- removed net N$35: R47.2, U8.QD
- removed net N$36: C19.2, R2.2, R7.1
- removed net N$37: C18.1, R7.2, U10A.+
- removed net N$38: R48.2, U8.QC
- removed net N$39: R49.2, U8.QA
- removed net N$40: C19.1, U1.VINR, U10A.-, U10A.OUT
- removed net N$41: C21.2, R8.2, R9.1
- removed net N$42: C20.1, R9.2, U10B.+
- removed net N$43: R45.1, U8.QB
- removed net N$44: C21.1, U1.VINL, U10B.-, U10B.OUT
- removed net N$45: C24.1, U9.VOUT_L
- removed net N$46: R17.2, TP31.P$1, U4B.OUT
- removed net N$47: C24.2, R11.2, R8.1
- removed net N$48: C23.2, R10.2, R2.1
- removed net N$49: R22.1, U9.BCK
- removed net N$50: R22.2, U9.DATA
- removed net N$51: R22.4, U9.SCK
- removed net N$52: R22.3, U9.LRCLK
- removed net N$53: C23.1, U9.VOUT_R
- removed net N$54: R16.1, U1.VOUTL, U4A.+
- removed net N$55: C38.2, C45.2, FB9.2, U11.VA-
- removed net N$56: C43.2, C46.2, FB10.2, U11.VA+
- removed net N$57: C44.2, FB11.1, U11.VD+
- removed net N$58: TP23.P$1, U12A.-, U12A.OUT
- removed net N$59: R29.2, R30.1, U12B.-
- removed net N$60: TP26.P$1, U13A.-, U13A.OUT
- removed net N$61: R31.1, U11.VOUTR, U13A.+
- removed net N$62: R31.2, R32.1, U13B.-
- removed net N$63: R32.2, TP28.P$1, U13B.OUT
- removed net N$64: C47.2, C54.2, FB12.1, U14.VCC
- removed net N$65: C48.2, C49.2, U14.VCOM
- removed net N$66: C51.2, R23.2, R24.1
- removed net N$67: C50.1, R24.2, U15A.+
- removed net N$68: C51.1, U11.VINR, U15A.-, U15A.OUT
- removed net N$69: C53.2, R25.2, R26.1
- removed net N$70: C52.1, R26.2, U15B.+
- removed net N$71: C53.1, U11.VINL, U15B.-, U15B.OUT
- removed net N$72: C57.1, U14.VOUT_L
- removed net N$73: R30.2, TP25.P$1, U12B.OUT
- removed net N$74: C57.2, R25.1, R28.2
- removed net N$75: C56.2, R23.1, R27.2
- removed net N$76: R33.1, U14.BCK
- removed net N$77: R33.2, U14.DATA
- removed net N$78: R33.4, U14.SCK
- removed net N$79: R33.3, U14.LRCLK
- removed net N$8: C11.2, C8.2, FB2.2, U1.VA-
- removed net N$80: C56.1, U14.VOUT_R
- removed net N$81: R29.1, U11.VOUTL, U12A.+
- removed net N$82: C64.2, C67.2, FB13.2, U16.VA-
- removed net N$83: C65.2, C68.2, FB14.2, U16.VA+
- removed net N$84: C66.2, FB15.1, U16.VD+
- removed net N$85: TP17.P$1, U17A.-, U17A.OUT
- removed net N$86: R40.2, R41.1, U17B.-
- removed net N$87: TP20.P$1, U18A.-, U18A.OUT
- removed net N$88: R42.1, U16.VOUTR, U18A.+
- removed net N$89: R42.2, R43.1, U18B.-
- removed net N$90: R43.2, TP22.P$1, U18B.OUT
- removed net N$91: C69.2, C76.2, FB16.1, U19.VCC
- removed net N$92: C70.2, C71.2, U19.VCOM
- removed net N$93: C73.2, R34.2, R35.1
- removed net N$94: C72.1, R35.2, U20A.+
- removed net N$95: C73.1, U16.VINR, U20A.-, U20A.OUT
- removed net N$96: C75.2, R36.2, R37.1
- removed net N$97: C74.1, R37.2, U20B.+
- removed net N$98: C75.1, U16.VINL, U20B.-, U20B.OUT
- removed net N$99: C78.1, U19.VOUT_L
- removed net OSD_DEBUG_USB_DM: U36.D-_IN, U3B.USB0_DM
- removed net OSD_DEBUG_USB_DP: U36.D+_IN, U3B.USB0_DP
- removed net OSD_DEBUG_USB_ID: CN6.ID, U3B.USB0_ID
- removed net OSD_FPGA_GPIO0: U3C.GPMC_A0, U6.B1_IO14
- removed net OSD_FPGA_GPIO1: U3C.GPMC_A1, U6.B1_IO12
- removed net OSD_FPGA_GPIO2: U3C.GPMC_A2, U6.B1_IO11
- removed net OSD_FPGA_GPIO3: U3C.GPMC_A3, U6.B2_IO5
- removed net OSD_FPGA_GPIO4: U3C.GPMC_A4, U6.B1_IO13
- removed net OSD_FPGA_GPIO5: U3C.GPMC_A9, U6.B2_IO9
- removed net OSD_FPGA_GPIO6: U3C.GPMC_A10, U6.B2_IO4
- removed net OSD_FPGA_GPIO7: U3C.GPMC_A11, U6.B2_IO8
- removed net OSD_SPI_CS_FPGA: U3C.SPI0_CS0, U6.B1_IO2
- removed net OSD_SPI_MISO: U3C.SPI0_D0, U6.B1_IO6
- removed net OSD_SPI_MOSI: U3C.SPI0_D1, U6.B1_IO7
- removed net OSD_SPI_SCLK: U3C.SPI0_SCLK, U6.B1_IO1
- removed net OSD_USB1_DM: U37.USB_UP_DN, U3B.USB1_DM
- removed net OSD_USB1_DP: U37.USB_UP_DP, U3B.USB1_DP
- removed net OSD_USB1_VBUS: R133.1, U3B.USB1_DRVVBUS, U3B.USB1_VBUS
- removed net PCM_I2S_BCLK_BB: U23.FUNC1, U6.B1_CLK0
- removed net PCM_I2S_BCLK_EXT: U24.FUNC1, U6.B2_IO28
- removed net PCM_I2S_DOUT_BB: U23.DOUT, U6.B1_IO24
- removed net PCM_I2S_DOUT_EXT: U24.DOUT, U6.B2_IO29
- removed net PCM_I2S_LRCLK_BB: U23.FUNC0, U6.B1_IO23
- removed net PCM_I2S_LRCLK_EXT: U24.FUNC0, U6.B2_IO31
- removed net PCM_I2S_MCLK_BB: U23.FUNC2, U6.B1_CLK1
- removed net PCM_I2S_MCLK_EXT: U24.FUNC2, U6.B2_CLK2
- removed net PGA0_!CS: U16.!CS, U6.B5_IO32
- removed net PGA0_!MUTE: U16.!MUTE, U6.B5_IO23
- removed net PGA0_SCLK: U16.SCLK, U6.B5_IO29
- removed net PGA0_SDI: U16.SDI, U6.B5_IO28
- removed net PGA1_!CS: U11.!CS, U6.B6_IO17
- removed net PGA1_!MUTE: U11.!MUTE, U6.B6_IO11
- removed net PGA1_SCLK: U11.SCLK, U6.B6_IO12
- removed net PGA1_SDI: U11.SDI, U6.B6_IO14
- removed net PGA2_!CS: U1.!CS, U6.B6_IO36
- removed net PGA2_!MUTE: U1.!MUTE, U6.B6_IO28
- removed net PGA2_SCLK: U1.SCLK, U6.B6_IO31
- removed net PGA2_SDI: U1.SDI, U6.B6_IO32
- removed net PSU_AMP_PWR_EN: Q1.G, R131.2, U6.B2_IO22
- removed net SHIFT_OUT: R112.2, U30.QH
- removed net UI_INPUT_AIRPLAY: R124.1, U6.B8_IO25
- removed net UI_INPUT_SEL: U45.Q, U6.B8_IO34
- removed net UI_INPUT_USB: R125.1, U6.B8_IO16
- removed net USB_OUT0_DN: U35.D-_IN, U37.USB_DN1_DN
- removed net USB_OUT0_DP: U35.D+_IN, U37.USB_DN1_DP
- removed net USB_OUT1_DN: R89.1, U37.USB_DN2_DN
- removed net USB_OUT1_DP: R88.1, U37.USB_DN2_DP
- removed net USB_RESET: U37.!RESET
- new net 12V: CN1.12V, CN4.1, U1.VIN+
- new net CM4_ENABLE: RPI-CM1G$1.GLOBAL_EN
- new net CM4_ETH_LED1: R3.2, RPI-CM1G$1.ETH_!LED1
- new net CM4_ETH_LED2: R4.2, RPI-CM1G$1.ETH_!LED2
- new net CM4_ETH_LED3: R5.2, RPI-CM1G$1.ETH_!LED3
- new net CM4_ETH_TRD0_N: CN3.TD0-, RPI-CM1G$1.ETH_PAIR0_N
- new net CM4_ETH_TRD0_P: CN3.TD0+, RPI-CM1G$1.ETH_PAIR0_P
- new net CM4_ETH_TRD1_N: CN3.TD1-, RPI-CM1G$1.ETH_PAIR1_N
- new net CM4_ETH_TRD1_P: CN3.TD1+, RPI-CM1G$1.ETH_PAIR1_P
- new net CM4_ETH_TRD2_N: CN3.TD2-, RPI-CM1G$1.ETH_PAIR2_N
- new net CM4_ETH_TRD2_P: CN3.TD2+, RPI-CM1G$1.ETH_PAIR2_P
- new net CM4_ETH_TRD3_N: CN3.TD3-, RPI-CM1G$1.ETH_PAIR3_N
- new net CM4_ETH_TRD3_P: CN3.TD3+, RPI-CM1G$1.ETH_PAIR3_P
- new net CM4_PCIE_CLK_N: CN1.REFCLK-, RPI-CM1G$2.PCIE_CLK_N
- new net CM4_PCIE_CLK_P: CN1.REFCLK+, RPI-CM1G$2.PCIE_CLK_P
- new net CM4_PCIE_CLK_REQ: CN1.!CLKREQ, RPI-CM1G$2.PCIE_CLK_!REQ
- new net CM4_PCIE_PCIE_RST: CN1.!PERST, RPI-CM1G$2.PCIE_!RST
- new net CM4_PCIE_RX_N: CN1.PERP0, RPI-CM1G$2.PCIE_RX_N
- new net CM4_PCIE_RX_P: CN1.PERN0, RPI-CM1G$2.PCIE_RX_P
- new net CM4_PCIE_TX_N: CN1.PETP0, RPI-CM1G$2.PCIE_TX_N
- new net CM4_PCIE_TX_P: CN1.PETN0, RPI-CM1G$2.PCIE_TX_P
- new net CM4_PI_ACT: R2.2, RPI-CM1G$1.PI_!LED_ACTIVITY
- new net CM4_PI_POWERED: R1.2, RPI-CM1G$1.PI_LED_!PWR
- new net CM4_PWR_1V8: RPI-CM1G$1.CM4_1.8V(OUTPUT)@88, RPI-CM1G$1.CM4_1.8V(OUTPUT)@90
- new net CM4_PWR_3V3: RPI-CM1G$1.CM4_3.3V(OUTPUT)@84, RPI-CM1G$1.CM4_3.3V(OUTPUT)@86, RPI-CM1G$1.GPIO_VREF
- new net CM4_RUN_PG: RPI-CM1G$1.RUN_PG
- new net CM4_USB_N: RPI-CM1G$2.USB_N, U2.D-_IN
- new net CM4_USB_P: RPI-CM1G$2.USB_P, U2.D+_IN
- net 3V3: now also CN1.!TRST, CN1.3V3, CN1.3V3AUX, CN1.TCK, CN1.TDI, CN1.TMS, U1.VO+; no longer C109.2, C110.2, C111.2, C112.2, C113.2, C114.2, C115.2, C116.2, C117.2, C118.2, C119.2, C120.2, C121.2, C125.2, C131.2, C151.2, C152.2, C153.2, C154.2, C155.2, C160.2, C161.2, C162.2, C163.2, C164.2, C2.2, C3.2, C30.2, C42.2, C5.2, C55.2, C6.2, C7.2, C85.2, C86.2, C87.2, C88.2, C92.2, C93.2, C94.2, C95.2, CN1.VCC, CN3.9, R1.2, R100.2, R106.2, R12.2, R122.2, R129.2, R15.2, R3.2, R54.2, R55.2, R56.2, R70.5, R70.6, R70.7, R70.8, R71.6, R71.7, R71.8, R72.2, R84.2, R85.2, R86.2, U22.!RESET, U22.VCC, U23.TEST, U23.VBUS, U23.VCCL, U23.VCCP, U23.VCCR, U23.VDD, U24.TEST, U24.VBUS, U24.VCCL, U24.VCCP, U24.VCCR, U24.VDD, U26.!RESET, U26.VCC, U30.!RESET, U30.VCC, U31.VCC, U37.VDD, U41.OUT, U41.OUT_S, U42.VCC, U43.VCC, U44.VCC, U45.VCC, U6.B1_NCONFIG, U6.VCCIO1, U6.VCCIO2, U6.VCCIO3, U6.VCCIO4, U6.VCCIO5, U6.VCCIO6, U6.VCCIO7, U6.VCCIO8, U8.!RESET, U8.VCC
- net 5V: now also CN2.VBUS, CN6.1, RPI-CM1G$1.+5V(INPUT)@77, RPI-CM1G$1.+5V(INPUT)@79, RPI-CM1G$1.+5V(INPUT)@81, RPI-CM1G$1.+5V(INPUT)@83, RPI-CM1G$1.+5V(INPUT)@85, RPI-CM1G$1.+5V(INPUT)@87, U2.VBUS; no longer C128.2, C130.A, FB11.2, FB15.2, FB7.2, R120.2, U1.ZCEN, U11.ZCEN, U16.ZCEN, U28.VOUT
- net GND: now also CN3.SHLD, CN5.1, RPI-CM1G$1.GND@1, RPI-CM1G$1.GND@13, RPI-CM1G$1.GND@14, RPI-CM1G$1.GND@2, RPI-CM1G$1.GND@22, RPI-CM1G$1.GND@23, RPI-CM1G$1.GND@32, RPI-CM1G$1.GND@33, RPI-CM1G$1.GND@42, RPI-CM1G$1.GND@43, RPI-CM1G$1.GND@52, RPI-CM1G$1.GND@53, RPI-CM1G$1.GND@59, RPI-CM1G$1.GND@60, RPI-CM1G$1.GND@65, RPI-CM1G$1.GND@66, RPI-CM1G$1.GND@7, RPI-CM1G$1.GND@71, RPI-CM1G$1.GND@74, RPI-CM1G$1.GND@8, RPI-CM1G$1.GND@98, RPI-CM1G$2.GND@107, RPI-CM1G$2.GND@108, RPI-CM1G$2.GND@113, RPI-CM1G$2.GND@114, RPI-CM1G$2.GND@119, RPI-CM1G$2.GND@120, RPI-CM1G$2.GND@125, RPI-CM1G$2.GND@126, RPI-CM1G$2.GND@131, RPI-CM1G$2.GND@132, RPI-CM1G$2.GND@137, RPI-CM1G$2.GND@138, RPI-CM1G$2.GND@144, RPI-CM1G$2.GND@150, RPI-CM1G$2.GND@155, RPI-CM1G$2.GND@156, RPI-CM1G$2.GND@161, RPI-CM1G$2.GND@162, RPI-CM1G$2.GND@167, RPI-CM1G$2.GND@168, RPI-CM1G$2.GND@173, RPI-CM1G$2.GND@174, RPI-CM1G$2.GND@179, RPI-CM1G$2.GND@180, RPI-CM1G$2.GND@185, RPI-CM1G$2.GND@186, RPI-CM1G$2.GND@191, RPI-CM1G$2.GND@192, RPI-CM1G$2.GND@197, RPI-CM1G$2.GND@198, RPI-CM1G$2.USB_OTG_ID, U1.COM, U1.VIN-, U2.GND; no longer C10.1, C100.1, C101.1, C102.1, C103.1, C104.1, C105.1, C106.1, C107.1, C108.1, C109.1, C110.1, C111.1, C112.1, C113.1, C114.1, C115.1, C116.1, C117.1, C118.1, C119.1, C120.1, C121.1, C122.1, C123.1, C124.1, C125.1, C127.1, C128.1, C129.K, C130.K, C131.1, C132.1, C133.1, C134.1, C135.1, C136.1, C137.1, C138.1, C139.1, C140.1, C141.1, C142.2, C143.1, C144.1, C145.1, C146.1, C148.1, C149.1, C150.1, C151.1, C152.1, C153.1, C154.1, C155.1, C156.1, C157.2, C158.1, C159.1, C160.1, C161.1, C162.1, C163.1, C164.1, C2.1, C29.1, C3.1, C30.1, C4.1, C42.1, C44.1, C5.1, C55.1, C6.1, C66.1, C7.1, C85.1, C86.1, C87.1, C88.1, C89.1, C90.1, C91.1, C92.1, C93.1, C94.1, C95.1, C96.1, C97.1, C98.1, C99.1, CN1.C_D2, CN3.10, CN3.6, CN4.GND, CN5.GND, CN6.GND, D10.A, D6.K, D7.A, D8.A, Q1.S, Q2.S, Q3.S, Q4.S, R104.1, R121.1, R127.1, R128.1, R130.1, R131.1, R132.1, R134.1, R135.1, R136.1, R137.1, R138.1, R14.1, R53.1, R57.1, R58.1, R59.1, R60.1, R61.1, R62.1, R63.1, R64.1, R65.1, R66.1, R67.1, R68.1, R69.1, R73.1, R90.1, RE1.GND, RE1.SW_B, SW1.2, TP1.P$1, TP6.P$1, TP9.P$1, U1.DGND, U11.DGND, U14.DEMP, U14.DGND, U14.FMT, U14.TEST, U16.DGND, U19.DEMP, U19.DGND, U19.FMT, U19.TEST, U21.K, U22.GND, U23.AGNDL, U23.AGNDR, U23.DGND, U23.FSEL, U23.FUNC3, U23.PGND, U23.PSEL, U23.ZGND, U24.AGNDL, U24.AGNDR, U24.DGND, U24.FSEL, U24.FUNC3, U24.PGND, U24.PSEL, U24.ZGND, U25.K, U26.GND, U29.K, U30.GND, U31.GND, U32.GND, U33.GND, U34.GND, U35.GND, U36.GND, U37.GND, U38.GND, U39.GND, U3B.USB1_ID, U3E.DGND@1, U3E.DGND@10, U3E.DGND@11, U3E.DGND@12, U3E.DGND@13, U3E.DGND@14, U3E.DGND@15, U3E.DGND@16, U3E.DGND@17, U3E.DGND@18, U3E.DGND@19, U3E.DGND@2, U3E.DGND@20, U3E.DGND@21, U3E.DGND@22, U3E.DGND@23, U3E.DGND@24, U3E.DGND@25, U3E.DGND@26, U3E.DGND@27, U3E.DGND@28, U3E.DGND@29, U3E.DGND@3, U3E.DGND@30, U3E.DGND@31, U3E.DGND@32, U3E.DGND@33, U3E.DGND@34, U3E.DGND@35, U3E.DGND@36, U3E.DGND@4, U3E.DGND@5, U3E.DGND@6, U3E.DGND@7, U3E.DGND@8, U3E.DGND@9, U40.AGND, U40.PGND, U41.AGND, U41.PGND, U42.GND, U43.GND, U44.GND, U45.GND, U6.B1_IO28, U6.B1_IO29, U6.B1_NCE, U6.B6_MSEL0, U6.B6_MSEL1, U6.B6_MSEL2, U6.B6_MSEL3, U6.GND, U6.GNDA1, U6.GNDA2, U6.GNDA3, U6.GNDA4, U7.K, U8.GND, U9.DEMP, U9.DGND, U9.FMT, U9.TEST, XTAL3.GND, XTAL4.GND
- net N$1: now also D1.A; no longer R4.1, RE1.A
- net N$2: now also CN2.D-, U2.D-OUT; no longer R3.1, R5.1, RE1.B
- net N$3: now also D2.A, R2.1; no longer R116.1, R117.2, U2.ADJ
- net N$4: now also CN2.D+, U2.D+_OUT; no longer C39.1, C40.K, FB3.2, U27.VIN
- net N$5: now also D3.A, R3.1; no longer R12.1, R13.2, RE1.SW_A
- net N$6: now also C1.2, CN3.CT0, CN3.CT1, CN3.CT2, CN3.CT3; no longer C31.2, C33.A, FB1.2, U2.VIN
- net N$7: now also D4.A, R4.1; no longer FB3.1, L2.2
- net N$9: now also D5.A, R5.1; no longer C12.2, C9.2, FB5.2, U1.VA+
Other:
- note added: "Mag Jack replacement WM10313-ND"

Commit message: DSP main board nearly done. All others have some changes not sure what
Parts:
- removed MECH5: 6mm x 3mm, MISC:MOUNTHOLE
- added R6: 10k, r_0603:CRCW060310K0FKTA
- added R7, R8: 10R, r_0603:CRCW060310R0FKTA
- C1: value 0.1uF 50V -> 1nF 2kV; device c_0603:CL10B104KB8NNWC -> CAPACITORS:C1812C102KGRACAUTO
- CN4, CN5, CN6: device CONNECTORs:PCB_TAB -> CONNECTORs:PCB_TAB_SMALL
Connections:
- removed net CM4_RUN_PG: RPI-CM1G$1.RUN_PG
- new net N$10: R7.2, RPI-CM1G$1.BT_!DISABLE
- new net N$11: R8.2, RPI-CM1G$1.WL_!DISABLE
- new net N$8: R6.2, RPI-CM1G$1.!RPIBOOT
- net CM4_PWR_3V3: now also R6.1
- net GND: now also R7.1, R8.1
Changed lines of the file:
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@@
 <part name="MECH3" library="MISC" deviceset="MOUNTHOLE" device="" value="6mm x 3mm"/>
 <part name="MECH4" library="MISC" deviceset="MOUNTHOLE" device="" value="6mm x 3mm"/>
-<part name="MECH5" library="MISC" deviceset="MOUNTHOLE" device="" value="6mm x 3mm"/>
 <part name="MECH6" library="MISC" deviceset="MOUNTHOLE" device="" value="6mm x 3mm"/>
 <part name="MECH7" library="MISC" deviceset="MOUNTHOLE" device="" value="6mm x 3mm"/>
@@
 <part name="CN2" library="CONNECTORs" deviceset="629104190121" device="" value="USB A"/>
 <part name="CN3" library="CONNECTORs" deviceset="0857931020" device="" value="Gb RJ45 + MAG"/>
-<part name="CN4" library="CONNECTORs" deviceset="PCB_TAB" device="" value="PCB Tab"/>
-<part name="CN5" library="CONNECTORs" deviceset="PCB_TAB" device="" value="PCB Tab"/>
-<part name="CN6" library="CONNECTORs" deviceset="PCB_TAB" device="" value="PCB Tab"/>
+<part name="CN4" library="CONNECTORs" deviceset="PCB_TAB_SMALL" device="" value="PCB Tab"/>
+<part name="CN5" library="CONNECTORs" deviceset="PCB_TAB_SMALL" device="" value="PCB Tab"/>
+<part name="CN6" library="CONNECTORs" deviceset="PCB_TAB_SMALL" device="" value="PCB Tab"/>
 <part name="U1" library="ICs" deviceset="PDQE15-Q24-S3-D" device="" value="DCDC 3V3"/>
 <part name="GND5" library="NETS" deviceset="GND" device=""/>
@@
 <part name="GND12" library="NETS" deviceset="GND" device=""/>
 <part name="GND13" library="NETS" deviceset="GND" device=""/>
-<part name="C1" library="c_0603" deviceset="CL10B104KB8NNWC" device="" value="0.1uF 50V"/>
+<part name="C1" library="CAPACITORS" deviceset="C1812C102KGRACAUTO" device="" value="1nF 2kV"/>
 <part name="GND14" library="NETS" deviceset="GND" device=""/>
+<part name="R6" library="r_0603" deviceset="CRCW060310K0FKTA" device="" value="10k"/>
+<part name="R7" library="r_0603" deviceset="CRCW060310R0FKTA" device="" value="10R"/>
+<part name="R8" library="r_0603" deviceset="CRCW060310R0FKTA" device="" value="10R"/>
 </parts>
 <sheets>
@@
 <attribute name="NAME" x="88.9" y="229.616" size="1.27" layer="95" align="center"/>
 </instance>
-<instance part="MECH5" gate="G$1" x="96.52" y="226.06" smashed="yes">
-<attribute name="NAME" x="96.52" y="229.616" size="1.27" layer="95" align="center"/>
-</instance>
 <instance part="MECH6" gate="G$1" x="104.14" y="226.06" smashed="yes">
 <attribute name="NAME" x="104.14" y="229.616" size="1.27" layer="95" align="center"/>
@@
 <instance part="GND14" gate="G$1" x="406.4" y="86.36" smashed="yes">
 <attribute name="VALUE" x="406.4" y="83.82" size="1.778" layer="96" align="center"/>
+</instance>
+<instance part="R6" gate="G$1" x="-7.62" y="33.02" smashed="yes">
+<attribute name="NAME" x="-7.62" y="35.56" size="1.27" layer="95" align="center"/>
+<attribute name="VALUE" x="-7.62" y="30.48" size="1.27" layer="96" align="center"/>
+</instance>
+<instance part="R7" gate="G$1" x="-2.54" y="38.1" smashed="yes">
+<attribute name="NAME" x="-2.54" y="40.64" size="1.27" layer="95" align="center"/>
+<attribute name="VALUE" x="-2.54" y="35.56" size="1.27" layer="96" align="center"/>
+</instance>
+<instance part="R8" gate="G$1" x="-7.62" y="43.18" smashed="yes">
+<attribute name="NAME" x="-7.62" y="45.72" size="1.27" layer="95" align="center"/>
+<attribute name="VALUE" x="-7.62" y="40.64" size="1.27" layer="96" align="center"/>
 </instance>
 </instances>
@@
 <wire x1="406.4" y1="88.9" x2="406.4" y2="91.44" width="0.1524" layer="91"/>
 </segment>
+<segment>
+<pinref part="R8" gate="G$1" pin="1"/>
+<wire x1="-12.7" y1="43.18" x2="-43.18" y2="43.18" width="0.1524" layer="91"/>
+<label x="-40.64" y="43.18" size="1.778" layer="95"/>
+</segment>
+<segment>
+<pinref part="R7" gate="G$1" pin="1"/>
+<wire x1="-7.62" y1="38.1" x2="-43.18" y2="38.1" width="0.1524" layer="91"/>
+<label x="-40.64" y="38.1" size="1.778" layer="95"/>
+</segment>
 </net>
 <net name="5V" class="0">
@@
 </segment>
 </net>
-<net name="CM4_RUN_PG" class="0">
-<segment>
-<pinref part="RPI-CM1" gate="G$1" pin="RUN_PG"/>
-<wire x1="129.54" y1="38.1" x2="170.18" y2="38.1" width="0.1524" layer="91"/>
-<label x="137.16" y="38.1" size="1.778" layer="95"/>
-</segment>
-</net>
 <net name="CM4_PWR_1V8" class="0">
 <segment>
@@
 <wire x1="129.54" y1="55.88" x2="170.18" y2="55.88" width="0.1524" layer="91"/>
 <label x="137.16" y="55.88" size="1.778" layer="95"/>
+</segment>
+<segment>
+<pinref part="R6" gate="G$1" pin="1"/>
+<label x="-40.64" y="33.02" size="1.778" layer="95"/>
+<wire x1="-12.7" y1="33.02" x2="-43.18" y2="33.02" width="0.1524" layer="91"/>
 </segment>
 </net>
@@
 </segment>
 </net>
+<net name="N$8" class="0">
+<segment>
+<pinref part="RPI-CM1" gate="G$1" pin="!RPIBOOT"/>
+<wire x1="68.58" y1="35.56" x2="2.54" y2="35.56" width="0.1524" layer="91"/>
+<wire x1="2.54" y1="35.56" x2="2.54" y2="33.02" width="0.1524" layer="91"/>
+<wire x1="2.54" y1="33.02" x2="-2.54" y2="33.02" width="0.1524" layer="91"/>
+<pinref part="R6" gate="G$1" pin="2"/>
+</segment>
+</net>
+<net name="N$10" class="0">
+<segment>
+<pinref part="R7" gate="G$1" pin="2"/>
+<pinref part="RPI-CM1" gate="G$1" pin="BT_!DISABLE"/>
+<wire x1="2.54" y1="38.1" x2="68.58" y2="38.1" width="0.1524" layer="91"/>
+</segment>
+</net>
+<net name="N$11" class="0">
+<segment>
+<pinref part="RPI-CM1" gate="G$1" pin="WL_!DISABLE"/>
+<wire x1="68.58" y1="40.64" x2="2.54" y2="40.64" width="0.1524" layer="91"/>
+<wire x1="2.54" y1="40.64" x2="2.54" y2="43.18" width="0.1524" layer="91"/>
+<pinref part="R8" gate="G$1" pin="2"/>
+<wire x1="2.54" y1="43.18" x2="-2.54" y2="43.18" width="0.1524" layer="91"/>
+</segment>
+</net>
