File: sa_amp.brd (EAGLE design)
At the start: 160 x 50 mm, 96 parts, among them CN1 PCB Tab, CN2 PCB Tab, CN3 PCB Tab, CN4 PCB Tab, CN5 PCB Tab, CN6 PCB Tab, CN7 TC2030, CN8 NO FIT, Q1 2N7002, U1 STM32L031G6, U2 15V REG, U3 LM7812, U4 TPA3255, U5 LM317

Commit message: Updated amplifier boards
Routing:
- net GND: track 220.3 -> 263.1 mm
- net RLY_EN: vias 2 -> 4
Changed lines of the file:
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@@
 </layers>
 <board>
-<fusionsync huburn="a.YnVzaW5lc3M6bXl1Y2wxNDk2" projecturn="a.YnVzaW5lc3M6bXl1Y2wxNDk2IzIwMjIwMjAyNDkyNTM5Mjc2" f3durn="urn:adsk.wipprod:dm.lineage:MC4icXcqTnGoFOp60mNzOw" pcbguid="" lastpulledtime="" lastsyncedchangeguid="f5b82504-2f50-8890-a936-34cf81d0887f" latestrevisionid="8ead1e05-3205-47fa-8a02-4f21de01c507" lastsyncedrevisionid="8ead1e05-3205-47fa-8a02-4f21de01c507" lastboardhashguid="6a9ea676-596f-2f4f-2220-b6cc05552d6a" lastpushedtime="2022-02-02T15:27:04Z" linktopcb3d="true"/>
+<fusionsync huburn="a.YnVzaW5lc3M6bXl1Y2wxNDk2" projecturn="a.YnVzaW5lc3M6bXl1Y2wxNDk2IzIwMjIwMjAyNDkyNTM5Mjc2" f3durn="urn:adsk.wipprod:dm.lineage:MC4icXcqTnGoFOp60mNzOw" pcbguid="" lastpulledtime="" lastsyncedchangeguid="f5b82504-2f50-8890-a936-34cf81d0887f" latestrevisionid="e5008f3a-a8c1-49bb-84f5-44e9d7aa8bfb" lastsyncedrevisionid="e5008f3a-a8c1-49bb-84f5-44e9d7aa8bfb" lastboardhashguid="60f55ca1-4b95-6ca5-7ac3-0c6fc0c5400c" lastpushedtime="2022-02-07T19:07:04Z" linktopcb3d="true"/>
 <plain>
 <wire x1="-47.5" y1="-22" x2="-44.5" y2="-25" width="0" layer="20" curve="90"/>
@@
 <contactref element="R59" pad="1"/>
 <polygon width="0.15" layer="2" isolate="0.15">
-<vertex x="-47.5" y="25"/>
+<vertex x="-16" y="25"/>
 <vertex x="112.5" y="25"/>
 <vertex x="112.5" y="-25"/>
-<vertex x="-47.5" y="-25"/>
+<vertex x="-39.25" y="-25"/>
+<vertex x="-39.25" y="-15.875"/>
+<vertex x="-29" y="-5.625"/>
+<vertex x="-29" y="0.625"/>
+<vertex x="-26.375" y="3.25"/>
+<vertex x="-21.25" y="3.25"/>
+<vertex x="-17.25" y="-0.75"/>
+<vertex x="-17.25" y="-5.625"/>
+<vertex x="-2.875" y="-5.625"/>
+<vertex x="-2.875" y="7.25"/>
+<vertex x="-16" y="7.25"/>
 </polygon>
 <wire x1="3.75" y1="0.3175" x2="2.6825" y2="0.3175" width="0.3" layer="16"/>
@@
 <wire x1="-23.375" y1="5.125" x2="-18.25" y2="5.125" width="0.15" layer="1"/>
 <wire x1="-38.375" y1="-7.5" x2="-25.75" y2="5.125" width="0.15" layer="16"/>
-<wire x1="-18.25" y1="5.125" x2="-16.375" y2="3.25" width="0.15" layer="1"/>
-<wire x1="-16.375" y1="3.25" x2="-8.625" y2="3.25" width="0.15" layer="1"/>
-<wire x1="-8.625" y1="3.25" x2="-7.875" y2="2.5" width="0.15" layer="1"/>
+<wire x1="-18.25" y1="5.125" x2="-15.625" y2="2.5" width="0.15" layer="1"/>
+<wire x1="-15.625" y1="2.5" x2="-7.875" y2="2.5" width="0.15" layer="1"/>
 <wire x1="-42.5" y1="7.5" x2="-34.625" y2="7.5" width="0.15" layer="1"/>
 <wire x1="-34.625" y1="7.5" x2="-33.75" y2="8.375" width="0.15" layer="1"/>
@@
 <wire x1="-5.25" y1="-4.375" x2="-4.8625" y2="-4.7625" width="0.15" layer="16"/>
 <polygon width="0.15" layer="3" isolate="0.15" rank="6">
-<vertex x="-47.5" y="25"/>
+<vertex x="-0.375" y="25"/>
 <vertex x="112.5" y="25"/>
 <vertex x="112.5" y="-25"/>
-<vertex x="-47.5" y="-25"/>
+<vertex x="-0.375" y="-25"/>
 </polygon>
 <contactref element="HOLE6" pad="1"/>
@@
 <via x="-38.125" y="-20.875" extent="1-16" drill="0.3"/>
 <contactref element="CN8" pad="3"/>
+<wire x1="-7.875" y1="5.375" x2="-7.875" y2="2.5" width="0.5" layer="1"/>
+<wire x1="-7.875" y1="2.5" x2="-7.875" y2="1.25" width="0.5" layer="1"/>
+<wire x1="-7.875" y1="1.25" x2="-7.875" y2="0" width="0.5" layer="1"/>
+<wire x1="-7.875" y1="0" x2="-7.875" y2="-1.25" width="0.5" layer="1"/>
+<wire x1="-7.875" y1="-1.25" x2="-7.875" y2="-2.5" width="0.5" layer="1"/>
+<wire x1="-7.875" y1="-2.5" x2="-7.875" y2="-9" width="0.5" layer="1"/>
+<wire x1="6.5" y1="-10.375" x2="9" y2="-7.875" width="0.5" layer="1"/>
+<wire x1="9" y1="-7.875" x2="15.875" y2="-7.875" width="0.5" layer="1"/>
+<wire x1="15.875" y1="-7.875" x2="18" y2="-10" width="0.5" layer="1"/>
+<wire x1="-7.875" y1="-9" x2="-6.5" y2="-10.375" width="0.5" layer="1"/>
+<wire x1="-6.5" y1="-10.375" x2="6.5" y2="-10.375" width="0.5" layer="1"/>
 </signal>
 <signal name="N$25">
@@
 <contactref element="U4" pad="38"/>
 <polygon width="0.15" layer="3" isolate="0.15" thermals="no">
-<vertex x="-31.25" y="7.25"/>
+<vertex x="-31.25" y="-5.625"/>
+<vertex x="-2.875" y="-5.625"/>
+<vertex x="-2.875" y="7.25"/>
 <vertex x="22.5" y="7.25"/>
 <vertex x="22.5" y="-25"/>
@@
 <wire x1="17.25" y1="23.5" x2="14.625" y2="20.875" width="0.15" layer="1"/>
 <wire x1="14.625" y1="20.875" x2="14.625" y2="14" width="0.15" layer="1"/>
-<wire x1="6.6875" y1="-4.8125" x2="0.125" y2="-11.375" width="0.15" layer="1"/>
+<wire x1="6.6875" y1="-4.8125" x2="1.875" y2="-9.625" width="0.15" layer="1"/>
+<wire x1="0.375" y1="-11.125" x2="0.125" y2="-11.375" width="0.15" layer="1"/>
 <wire x1="6.6875" y1="-4.8125" x2="6.6875" y2="6.0625" width="0.15" layer="1"/>
 <wire x1="6.6875" y1="6.0625" x2="14.625" y2="14" width="0.15" layer="1"/>
@@
 <contactref element="U1" pad="24"/>
 <wire x1="-20.875" y1="-13.5" x2="-20.875" y2="-14.85" width="0.15" layer="16"/>
+<via x="0.375" y="-11.125" extent="1-16" drill="0.3"/>
+<wire x1="0.375" y1="-11.125" x2="1.875" y2="-9.625" width="0.15" layer="16"/>
+<via x="1.875" y="-9.625" extent="1-16" drill="0.3"/>
 </signal>
 <signal name="N$8">
@@
 <mfgpreviewcolor name="silkscreencolor" color="0xFFFEFEFE"/>
 <mfgpreviewcolor name="backgroundcolor" color="0xFF282828"/>
-<mfgpreviewcolor name="coppercolor" color="0xFFFFBF00"/>
+<mfgpreviewcolor name="coppercolor" color="0xFF858585"/>
 <mfgpreviewcolor name="substratecolor" color="0xFF282828"/>
 </mfgpreviewcolors>
